File: platform/mains-protection/hw/mains-protection-panel.sch (EAGLE design)
At the start: 29 parts, among them IC1 MEGA8-P

Commit message: enabling main features
Other:
- note added: "LED is moved to PD3+PD4 to free up serial port"
Changed lines of the file:
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@@
 <text x="83.82" y="66.04" size="2.54" layer="94">Calculate values of resistors according to the desired brightness</text>
 <text x="119.38" y="142.24" size="2.54" layer="94">The firmware is for ATMEGA48</text>
+<text x="165.1" y="114.3" size="1.778" layer="94">LED is moved to PD3+PD4 to free up serial port</text>
 </plain>
 <instances>
