File: target/roller-shutter-controller/hardware/roller-shutter-controller.brd (EAGLE design)
At the start: 40 x 50 mm, 41 parts, among them IC1 MEGA48-AI, J1 AVRISP6, Q1 4 MHz, T1 BTA600, T2 BTA600, U1 MCP2510SO, U2 MCP2551SN, X1 MCV2, X2 MCV2, X3 MCV2, X4 MKDSN1,5/2-5,08, X5 MKDSN1,5/2-5,08, X6 MCV2

Commit message: fixes
Parts:
- added R10: 20k, rcl:R0805
- moved R9 4.27 mm to (21.1, 26.5)
- moved C8 0.24 mm to (12.0, 20.8)
Connections:
- removed net VCC: J1.2
- new net N$19: R10.1, U1.17
- net VDD: now also J1.2, R10.2
Routing:
- net VDD: track 99.8 -> 108.8 mm, vias 2 -> 4
- net N$19: track 0.00 -> 5.22 mm
- net L2: track 11.5 -> 6.57 mm
- net INT: track 36.3 -> 40.2 mm
- net N$18: track 8.86 -> 12.2 mm

Commit message: roller-shutter-controller: improved board
Parts:
- added LED1: (no value), led:CHIP-LED0805
- added PAD6, PAD7: (no value), wirepad:1,6/0,8
- added R11: 20k, rcl:R0805
- C1: value (none) -> 220nF 50V
- moved C8 1.80 mm to (10.8, 22.1), turned to 270 degrees
- moved R10 0.91 mm to (16.2, 21.5), turned to 90 degrees
Connections:
- new net N$20: LED1.A, R11.2
- net INT: now also LED1.C
- net VDD: now also PAD6.1, R11.1
- net VSS: now also PAD7.1
Routing:
- net INT: track 40.2 -> 51.5 mm
- net VDD: track 108.8 -> 106.5 mm
- net N$20: track 0.00 -> 2.35 mm
- net VSS: track 222.2 -> 221.1 mm
- net N$19: track 5.22 -> 4.42 mm
