File: target/roller-shutter-controller/hardware/roller-shutter-controller.sch (EAGLE design)
At the start: 41 parts, among them IC1 MEGA48-AI, J1 AVRISP6, Q1 4 MHz, T1 BTA600, T2 BTA600, U1 MCP2510SO, U2 MCP2551SN, X1 MCV2, X2 MCV2, X3 MCV2, X4 MKDSN1,5/2-5,08, X5 MKDSN1,5/2-5,08, X6 MCV2

Commit message: fixes
Parts:
- added R10: 20k, rcl:R-EU_R0805
Connections:
- new net N$19: R10.1, U1>NAME.RESET
- net VDD: now also J1.VCC, R10.2
Changed lines of the file:
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@@
 <setting verticaltext="up"/>
 </settings>
-<grid distance="0.25" unitdist="inch" unit="inch" style="lines" multiple="1" display="yes" altdistance="0.01" altunitdist="inch" altunit="inch"/>
+<grid distance="0.1" unitdist="inch" unit="inch" style="lines" multiple="1" display="no" altdistance="0.01" altunitdist="inch" altunit="inch"/>
 <layers>
 <layer number="1" name="Top" color="4" fill="1" visible="no" active="no"/>
@@
 <part name="R8" library="rcl" deviceset="R-EU_" device="R0805" value="10.2k"/>
 <part name="R9" library="rcl" deviceset="R-EU_" device="R0805" value="10.2k"/>
+<part name="R10" library="rcl" deviceset="R-EU_" device="R0805" value="20k"/>
 </parts>
 <sheets>
@@
 <instance part="R8" gate="G$1" x="154.94" y="167.64"/>
 <instance part="R9" gate="G$1" x="154.94" y="132.08"/>
+<instance part="R10" gate="G$1" x="160.02" y="71.12" rot="R180"/>
 </instances>
 <busses>
@@
 <label x="144.78" y="68.58" size="1.778" layer="95" rot="R90"/>
 </segment>
+<segment>
+<pinref part="J1" gate="A" pin="VCC"/>
+<wire x1="48.26" y1="27.94" x2="40.64" y2="27.94" width="0.1524" layer="91"/>
+<label x="40.64" y="27.94" size="1.778" layer="95"/>
+</segment>
+<segment>
+<pinref part="R10" gate="G$1" pin="2"/>
+<wire x1="154.94" y1="71.12" x2="147.32" y2="71.12" width="0.1524" layer="91"/>
+<label x="147.32" y="71.12" size="1.778" layer="95"/>
+</segment>
 </net>
 <net name="LX" class="0">
@@
 </segment>
 </net>
+<net name="N$19" class="0">
+<segment>
+<pinref part="U1" gate="&gt;NAME" pin="RESET"/>
+<pinref part="R10" gate="G$1" pin="1"/>
+</segment>
+</net>

Commit message: roller-shutter-controller: improved board
Parts:
- added LED1: (no value), led:LEDCHIP-LED0805
- added PAD6, PAD7: (no value), wirepad:1,6/0,8
- added R11: 20k, rcl:R-EU_R0805
- C1: value (none) -> 220nF 50V
Connections:
- new net N$20: LED1.A, R11.2
- net INT: now also LED1.C
- net VDD: now also PAD6.P, R11.1
- net VSS: now also PAD7.P
Changed lines of the file:
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@@
 <part name="X2" library="con-phoenix-381_l" deviceset="MCV2" device=""/>
 <part name="U$1" library="my-allegro" deviceset="A8499SLJT" device="" value="A8499"/>
-<part name="C1" library="rcl" deviceset="C-EU" device="C0805"/>
+<part name="C1" library="rcl" deviceset="C-EU" device="C0805" value="220nF 50V"/>
 <part name="C2" library="rcl" deviceset="CPOL-EU" device="153CLV-1010" value="100uF 63V"/>
 <part name="R5" library="rcl" deviceset="R-EU_" device="R0805" value="15k"/>
@@
 <part name="R9" library="rcl" deviceset="R-EU_" device="R0805" value="10.2k"/>
 <part name="R10" library="rcl" deviceset="R-EU_" device="R0805" value="20k"/>
+<part name="PAD6" library="wirepad" deviceset="1,6/0,8" device=""/>
+<part name="LED1" library="led" deviceset="LED" device="CHIP-LED0805"/>
+<part name="R11" library="rcl" deviceset="R-EU_" device="R0805" value="20k"/>
+<part name="PAD7" library="wirepad" deviceset="1,6/0,8" device=""/>
 </parts>
 <sheets>
@@
 <instance part="R9" gate="G$1" x="154.94" y="132.08"/>
 <instance part="R10" gate="G$1" x="160.02" y="71.12" rot="R180"/>
+<instance part="PAD6" gate="P" x="111.76" y="55.88" rot="R180"/>
+<instance part="LED1" gate="G$1" x="254" y="76.2"/>
+<instance part="R11" gate="G$1" x="254" y="83.82" rot="R270"/>
+<instance part="PAD7" gate="P" x="99.06" y="63.5"/>
 </instances>
 <busses>
@@
 <wire x1="109.22" y1="63.5" x2="101.6" y2="63.5" width="0.1524" layer="91"/>
 <label x="101.6" y="63.5" size="1.778" layer="95"/>
+<pinref part="PAD7" gate="P" pin="P"/>
 </segment>
 <segment>
@@
 <label x="147.32" y="71.12" size="1.778" layer="95"/>
 </segment>
+<segment>
+<pinref part="PAD6" gate="P" pin="P"/>
+<wire x1="109.22" y1="55.88" x2="101.6" y2="55.88" width="0.1524" layer="91"/>
+<label x="101.6" y="55.88" size="1.778" layer="95"/>
+</segment>
+<segment>
+<pinref part="R11" gate="G$1" pin="1"/>
+<wire x1="254" y1="88.9" x2="254" y2="96.52" width="0.1524" layer="91"/>
+<label x="254" y="91.44" size="1.778" layer="95" rot="R90"/>
+</segment>
 </net>
 <net name="LX" class="0">
@@
 <label x="200.66" y="71.12" size="1.778" layer="95"/>
 </segment>
+<segment>
+<pinref part="LED1" gate="G$1" pin="C"/>
+<wire x1="254" y1="71.12" x2="254" y2="63.5" width="0.1524" layer="91"/>
+<label x="254" y="63.5" size="1.778" layer="95" rot="R90"/>
+</segment>
 </net>
 <net name="N$13" class="0">
@@
 </segment>
 </net>
+<net name="N$20" class="0">
+<segment>
+<pinref part="R11" gate="G$1" pin="2"/>
+<pinref part="LED1" gate="G$1" pin="A"/>
+</segment>
+</net>
