File: target/wr703n-display/hardware/wr703n-display.brd (EAGLE design)
At the start: 24 parts, among them IC1 MEGA48-AI, J2 22-05-7048-04, J3 22-05-7028-02

Commit message: wr703n-display
Parts:
- added R1: 330, rcl:R0805
- added TP16, TP17, TP18: PTR1B2,54, testpad:B2,54
- moved TP6 24.4 mm to (11.4, 38.1)
- moved TP13 6.70 mm to (19.4, 23.5)
- moved TP5 5.24 mm to (36.8, 30.5)
- moved TP1 4.07 mm to (12.1, 25.4)
- moved TP2 3.81 mm to (6.35, 45.7)
- moved TP10 3.81 mm to (33.0, 41.9)
- moved TP11 3.81 mm to (33.0, 39.4)
- moved TP12 3.81 mm to (38.1, 39.4)
- moved TP7 3.81 mm to (38.1, 41.9)
- moved TP8 3.81 mm to (35.6, 41.9)
- moved TP9 3.81 mm to (35.6, 39.4)
- moved C7 2.54 mm to (28.3, 26.5)
- moved TP14 2.54 mm to (22.2, 23.5)
- moved TP4 2.54 mm to (14.6, 33.0)
- moved C1 2.54 mm to (15.2, 38.4)
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Connections:
- new net PB1: IC1.13, R1.1
- net LED: now also R1.2; no longer IC1.13
- net VSS: now also TP16.TP, TP17.TP, TP18.TP
Routing:
- net LED: track 18.6 -> 8.99 mm
- net VSS: track 108.5 -> 115.2 mm
- net N$7: track 9.81 -> 3.60 mm
- net VDD: track 33.2 -> 39.3 mm
- net PB1: track 0.00 -> 5.13 mm
- net RESET: track 42.0 -> 37.7 mm
- net N$6: track 4.34 -> 8.52 mm
- net SCL: track 15.9 -> 13.2 mm
- net SCE: track 22.1 -> 19.6 mm
- net RST: track 15.4 -> 12.9 mm
- net DI: track 15.8 -> 13.3 mm
- net SCLK: track 17.2 -> 14.6 mm
- net DC: track 15.5 -> 12.9 mm
- net N$3: track 8.62 -> 6.88 mm
- net SDA: track 14.9 -> 13.3 mm
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