File: target/lcd20x4/hardware/lcd20x4_left.brd (EAGLE design)
At the start: 100 x 80 mm, 57 parts, among them IC1 LTC485N, IC2 MC34063AD

Commit message: lcd20x4_leds
Routing:
- net RS485_A: track 51.3 -> 43.6 mm
- net GND: track 337.0 -> 341.3 mm, vias 4 -> 7
- net VBUS: track 38.3 -> 41.4 mm, vias 0 -> 3
- net RS485_B: track 49.6 -> 48.7 mm
- net VCC: track 316.9 -> 317.8 mm
- net OW: track 31.8 -> 32.0 mm, vias 0 -> 1
Other:
- board size 100 x 80 mm -> 100 x 61 mm
