File: target/eprom-programmer/hardware/eprom-programmer3.sch (EAGLE design)
At the start: 42 parts, among them IC2 27C08032P6, Q1 BC557, Q2 BC557, Q3 BC557

Commit message: eprom-programmer: hardware
Parts:
- added R10, R9: 5k1, rcl:R-EU_M0805
Connections:
- new net N$11: Q1.B, R9.1
- new net N$14: Q2.B, R10.1
- net N$2: now also R10.2; no longer Q2.B
- net N$4: now also R9.2; no longer Q1.B
Other:
- moved on the sheet: C1, C2, D1, IC2, JP1, JP2, JP3, JP4, LED1, PAD1, PAD10, PAD11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
