File: target/button-led-matrix-4x4/hardware/button-led-matrix-4x4.sch (EAGLE design)
At the start: 23 parts, among them IC1 ATMEGA48/88/168-AU, X1 CRYSTALS-NOGND-HC49

Commit message: button-led-matrix-4x4 hardware
Parts:
- added C3, C4: 18, rcl:C-EUC0805
- added IC2: AMS1117-3.3, burr-brown:REG1117
- added PAD10, PAD100, PAD101, PAD102, PAD103, PAD104, PAD105, PAD11, PAD12, PAD13, PAD14, PAD15, PAD16, PAD17, PAD18, PAD19, PAD20, PAD21, PAD22, PAD23, PAD24, PAD25, PAD26, PAD27, PAD28, PAD29, PAD3, PAD30, PAD31, PAD32, PAD33, PAD34, PAD35, PAD36, PAD37, PAD38, PAD39, PAD4, PAD40, PAD41, PAD42, PAD43, PAD44, PAD45, PAD46, PAD47, PAD48, PAD49, PAD5, PAD50, PAD51, PAD52, PAD53, PAD54, PAD55, PAD56, PAD57, PAD58, PAD59, PAD6, PAD60, PAD61, PAD62, PAD63, PAD64, PAD65, PAD66, PAD67, PAD68, PAD69, PAD7, PAD70, PAD71, PAD72, PAD73, PAD74, PAD75, PAD76, PAD77, PAD78, PAD79, PAD8, PAD80, PAD81, PAD82, PAD83, PAD84, PAD85, PAD86, PAD87, PAD89, PAD9, PAD90, PAD91, PAD92, PAD93, PAD94, PAD95, PAD96, PAD97, PAD98, PAD99: WIREPADSMD1,27-254, wirepad:WIREPADSMD1,27-254
- added PAD88: (no value), wirepad:1,6/0,8
- added R1, R2: (no value), rcl:R-EU_R1206
- added R3, R4: (no value), rcl:R-EU_R0805
Connections:
- removed net N$11: IC1.PD5(T1/OC0B/PCINT21)
- removed net N$13: IC1.PD7(AIN1/PCINT23)
- removed net N$14: IC1.PB0(ICP1/CLKO/PCINT0)
- removed net N$15: IC1.PB1(OC1A/PCINT1)
- removed net N$16: IC1.PB2(SS/OC1B/PCINT2)
- removed net N$18: IC1.PB4(MISO/PCINT4)
- removed net N$19: IC1.PB5(SCK/PCINT5)
- removed net N$32: S1G$3.SIG2
- removed net N$65: LED5.GND
- removed net N$66: LED6.GND
- removed net N$67: LED7.GND
- removed net N$68: LED8.GND
- removed net N$7: IC1.PD0(RXD/PCINT16)
- removed net N$9: IC1.PD3(INT1/OC2B/PCINT19)
- new net INT: IC1.PD0(RXD/PCINT16), PAD67.P, PAD68.P, PAD69.P, PAD70.P, PAD71.P, PAD72.P, PAD92.P
- new net N$17: PAD98.P, R4.2
- new net N$20: PAD79.P
- new net XTAL1: C4.2, IC1.PB6(XTAL1/TOSC1/PCINT6), X1.2
- new net XTAL2: C3.2, IC1.PB7(XTAL2/TOSC2/PCINT7), X1.1
- net B1: now also IC1.PD4(T0/XCK/PCINT20), PAD18.P, PAD89.P
- net B10: now also IC1.PC1(ADC1/PCINT9), PAD23.P, PAD32.P
- net B11: now also IC1.PB5(SCK/PCINT5), PAD25.P, PAD33.P
- net B12: now also IC1.PB1(OC1A/PCINT1), PAD28.P, PAD34.P
- net B13: now also IC1.PC2(ADC2/PCINT10), PAD12.P, PAD38.P
- net B14: now also IC1.PC0(ADC0/PCINT8), PAD24.P, PAD37.P
- net B15: now also IC1.PB4(MISO/PCINT4), PAD26.P, PAD36.P
- net B16: now also IC1.PB2(SS/OC1B/PCINT2), PAD27.P, PAD35.P
- net B2: now also IC1.PD5(T1/OC0B/PCINT21), PAD13.P, PAD17.P
- net B3: now also IC1.PD6(AIN0/OC0A/PCINT22), PAD15.P
- net B4: now also IC1.PD7(AIN1/PCINT23), PAD16.P, PAD30.P
- net B5: now also IC1.PD3(INT1/OC2B/PCINT19), PAD103.P, R2.2, R4.1
- net B6: now also IC1.PD2(INT0/PCINT18), PAD102.P, R1.2, R3.1
- net B8: now also IC1.PB0(ICP1/CLKO/PCINT0), PAD29.P
- net B9: now also IC1.PC3(ADC3/PCINT11), PAD11.P, PAD31.P
- net DATA: now also PAD100.P, PAD101.P, PAD7.P
- net DO12: now also PAD10.P, PAD5.P
- net DO4: now also PAD3.P, PAD8.P
- net DO8: now also PAD4.P, PAD9.P
- net D_OUT: now also PAD6.P
- net GND: now also C3.1, C4.1, IC2.GND, LED5.GND, LED6.GND, LED7.GND, LED8.GND, PAD105.P, PAD44.P, PAD45.P, PAD50.P, PAD53.P, PAD58.P, PAD61.P, PAD65.P, PAD75.P, PAD87.P, PAD93.P, PAD95.P, S1G$3.SIG2
- net N$1: now also PAD86.P; no longer IC1.PB6(XTAL1/TOSC1/PCINT6), X1.2
- net N$10: now also PAD99.P; no longer IC1.PD4(T0/XCK/PCINT20)
- net N$12: now also PAD47.P; no longer IC1.PD6(AIN0/OC0A/PCINT22)
- net N$2: now also PAD97.P, R3.2; no longer IC1.PB7(XTAL2/TOSC2/PCINT7), X1.1
- net N$3: now also PAD19.P, PAD39.P; no longer IC1.PC0(ADC0/PCINT8)
- net N$4: now also PAD20.P, PAD40.P; no longer IC1.PC1(ADC1/PCINT9)
- net N$5: now also PAD21.P, PAD41.P; no longer IC1.PC2(ADC2/PCINT10)
- net N$6: now also PAD22.P, PAD42.P; no longer IC1.PC3(ADC3/PCINT11)
- net N$8: now also PAD43.P; no longer IC1.PD2(INT0/PCINT18)
- net RESET: now also PAD88.P
- net SCL: now also PAD51.P, PAD56.P, PAD60.P, PAD64.P, PAD73.P, PAD82.P, PAD91.P, R1.1
- net SDA: now also PAD52.P, PAD55.P, PAD59.P, PAD63.P, PAD74.P, PAD81.P, PAD90.P, R2.1
- net VCC: now also IC2.VIN, IC2.VOUT, PAD104.P, PAD46.P, PAD48.P, PAD49.P, PAD54.P, PAD57.P, PAD62.P, PAD66.P, PAD76.P, PAD83.P, PAD94.P, PAD96.P
Other:
- moved on the sheet: C1, C2, IC1, PAD1, PAD2, X1

Commit message: button-led-matrix-4x4 v1.1
Parts:
- added C10, C11, C12, C13, C14, C15, C16, C17, C18, C19, C5, C6, C7, C8, C9: 0.1, rcl:C-EUC0805
- added PAD106, PAD107, PAD108, PAD109: WIREPADSMD1,27-254, wirepad:WIREPADSMD1,27-254
Connections:
- net DO10: now also PAD106.P, PAD107.P
- net DO14: now also PAD108.P, PAD109.P
- net GND: now also C10.2, C11.2, C12.2, C13.2, C14.2, C15.2, C16.2, C17.2, C18.2, C19.2, C5.2, C6.2, C7.2, C8.2, C9.2
- net VCC: now also C10.1, C11.1, C12.1, C13.1, C14.1, C15.1, C16.1, C17.1, C18.1, C19.1, C5.1, C6.1, C7.1, C8.1, C9.1
