File: target/seq__control_pad/hardware/seq__control_pad_03.sch (EAGLE design)
At the start: 78 parts, among them IC1 MEGA48/88/168-AU, SW1 EC12E_SW

Commit message: seq__control_pad: hardware
Parts:
- added C1, C2: 0.1, rcl:C-EUC0805
- added C3, C4: 18pF, rcl:C-EUC0805
- added D12, D13, D14, D15, D16, D17, D18: (no value), diode:DIODE-MINIMELF
- added LD1: (no value), led:DUOLED-RY-A
- added PAD47, PAD48, PAD49, PAD50, PAD51, PAD52, PAD53, PAD54: WIREPAD1,6/0,8, wirepad:WIREPAD1,6/0,8
- added R1, R2, R3, R4, R5, R6, R7, R8, R9: (no value), rcl:R-EU_R0805
- added T1, T2, T3, T4: (no value), transistor:MMBT3904LT1-NPN-SOT23-BEC
Connections:
- removed net N$25: IC1.PB5(SCK/PCINT5)
- removed net N$30: IC1.PD7(AIN1/PCINT23)
- removed net N$31: IC1.PD5(T1/OC0B/PCINT21)
- removed net N$32: IC1.PD6(AIN0/OC0A/PCINT22)
- new net ADC6: IC1.ADC6, PAD49.P
- new net ADC7: IC1.ADC7, PAD48.P
- new net C0SEL: IC1.PC3(ADC3/PCINT11), R4.1
- new net C1SEL: IC1.PC0(ADC0/PCINT8), R1.1
- new net C2SEL: IC1.PC1(ADC1/PCINT9), R2.1
- new net C3SEL: IC1.PC2(ADC2/PCINT10), R3.1
- new net EA: IC1.PD6(AIN0/OC0A/PCINT22), SW1G$1.A
- new net EB: IC1.PD5(T1/OC0B/PCINT21), SW1G$1.B
- new net ES: IC1.PD7(AIN1/PCINT23), SW1G$2.2
- new net GND: C1.2, C2.2, C3.1, C4.1, IC1.AGND, IC1.GND@1, IC1.GND@2, PAD53.P, SW1G$1.C, SW1G$2.1, T1.E, T2.E, T3.E, T4.E
- new net INT: IC1.PB5(SCK/PCINT5), PAD54.P
- new net N$1: D11.C, S11.P
- new net N$20: D13.C, S15.P
- new net N$21: D14.C, S17.P
- new net N$23: D15.C, S12.S
- new net O0: IC1.PB4(MISO/PCINT4), R5.1
- new net O1: IC1.PB3(MOSI/OC2A/PCINT3), R6.1
- new net O2: IC1.PB2(SS/OC1B/PCINT2), R7.1
- new net O3: IC1.PB1(OC1A/PCINT1), R8.1
- new net O4: IC1.PB0(ICP1/CLKO/PCINT0), R9.1
- new net RESET: IC1.PC6(/RESET/PCINT14), PAD47.P
- new net SCL: IC1.PC5(ADC5/SCL/PCINT13), PAD51.P
- new net SDA: IC1.PC4(ADC4/SDA/PCINT12), PAD50.P
- new net VCC: C1.1, C2.1, IC1.AREF, IC1.AVCC, IC1.VCC@1, IC1.VCC@2, PAD52.P
- net C0: now also T4.C; no longer IC1.PC0(ADC0/PCINT8)
- net C1: now also T1.C
- net C2: now also LD1.CY, S11.S, S13.S, S15.S, S17.S, T2.C; no longer S11.P
- net C3: now also LD1.CR, S12.P1, S14.P1, S16.P1, S18.P1, T3.C
- net IR0: now also D15.A
- net IR1: now also D12.A, D16.A
- net IR2: now also D13.A, D17.A
- net IR3: now also D14.A, D18.A
- net N$19: now also D12.C, S13.P; no longer D11.C, S11.S
- net N$2: now also R1.2, T1.B; no longer IC1.PC1(ADC1/PCINT9)
- net N$3: now also R2.2, T2.B; no longer IC1.PC2(ADC2/PCINT10)
- net N$4: now also R3.2, T3.B; no longer IC1.PC3(ADC3/PCINT11)
- net N$6: now also D16.C, S14.S; no longer IC1.PC4(ADC4/SDA/PCINT12)
- net N$7: now also R4.2, T4.B; no longer IC1.PC5(ADC5/SCL/PCINT13)
- net N$8: now also D17.C, S16.S; no longer IC1.ADC6
- net N$9: now also D18.C, S18.S; no longer IC1.ADC7
- net OR0: now also R5.2; no longer IC1.PB4(MISO/PCINT4)
- net OR1: now also R6.2; no longer IC1.PB3(MOSI/OC2A/PCINT3)
- net OR2: now also R7.2; no longer IC1.PB2(SS/OC1B/PCINT2)
- net OR3: now also R8.2; no longer IC1.PB1(OC1A/PCINT1)
- net OR4: now also LD1.A, R9.2; no longer IC1.PB0(ICP1/CLKO/PCINT0)
- net XTAL1: now also C4.2
- net XTAL2: now also C3.2
Other:
- moved on the sheet: D11, SW1
