File: target/arduino_encoder_tester/hardware/arduino-shield.brd (EAGLE design)
At the start: 5 parts, among them SW1 EC12E_SW

Commit message: seq_blm update
Parts:
- added R2, R3: (no value), rcl:R0805
Connections:
- net SCL: now also R3.1
- net SDA: now also R2.1
- net VCC: now also R2.2, R3.2
Routing:
- net D: track 41.5 -> 60.4 mm
- net SDA: track 12.5 -> 15.4 mm
- net SCL: track 6.13 -> 8.95 mm
- net VCC: track 83.8 -> 83.1 mm
Changed lines of the file:
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@@
 </element>
 <element name="R1" library="rcl" package="R0805" value="" x="25.625" y="23.225" rot="R180"/>
+<element name="R2" library="rcl" package="R0805" value="" x="67.8975" y="14.085" rot="R90"/>
+<element name="R3" library="rcl" package="R0805" value="" x="65.185" y="14.125" rot="R90"/>
 </elements>
 <signals>
@@
 <wire x1="47.5" y1="5.36" x2="47.43" y2="5.29" width="1.27" layer="1"/>
 <polygon width="0.254" layer="1" isolate="0.6096" orphans="yes">
-<vertex x="22.86" y="2.54"/>
-<vertex x="69.85" y="2.54"/>
-<vertex x="69.85" y="55.88"/>
-<vertex x="22.86" y="55.88"/>
+<vertex x="0" y="-3.81"/>
+<vertex x="76.2" y="-3.81"/>
+<vertex x="76.2" y="58.42"/>
+<vertex x="0" y="58.42"/>
 </polygon>
 </signal>
@@
 <contactref element="U$1" pad="3V"/>
 <wire x1="39.81" y1="5.29" x2="39.81" y2="7.18" width="1.27" layer="1"/>
-<wire x1="39.81" y1="7.18" x2="39.37" y2="7.62" width="1.27" layer="1"/>
-<wire x1="39.37" y1="7.62" x2="24.13" y2="7.62" width="1.27" layer="1"/>
-<wire x1="24.13" y1="7.62" x2="24.13" y2="22.86" width="1.27" layer="1"/>
 <wire x1="24.13" y1="22.86" x2="24.13" y2="25.4" width="1.27" layer="1"/>
 <wire x1="28.38" y1="25.6275" x2="24.3575" y2="25.6275" width="1.27" layer="1"/>
@@
 <wire x1="39.37" y1="15.24" x2="28.9825" y2="25.6275" width="1.27" layer="1"/>
 <wire x1="28.9825" y1="25.6275" x2="28.38" y2="25.6275" width="1.27" layer="1"/>
+<contactref element="R2" pad="2"/>
+<contactref element="R3" pad="2"/>
+<wire x1="67.8975" y1="15.035" x2="67.6925" y2="15.24" width="1.27" layer="1"/>
+<wire x1="67.6925" y1="15.24" x2="65.35" y2="15.24" width="1.27" layer="1"/>
+<wire x1="65.35" y1="15.24" x2="62.23" y2="15.24" width="1.27" layer="1"/>
+<wire x1="65.185" y1="15.075" x2="65.35" y2="15.24" width="1.27" layer="1"/>
+<wire x1="24.13" y1="22.86" x2="24.13" y2="19.05" width="1.27" layer="1"/>
+<wire x1="24.13" y1="19.05" x2="25.4" y2="17.78" width="1.27" layer="1"/>
+<wire x1="25.4" y1="17.78" x2="29.21" y2="17.78" width="1.27" layer="1"/>
+<wire x1="29.21" y1="17.78" x2="39.81" y2="7.18" width="1.27" layer="1"/>
 </signal>
 <signal name="LIGHT">
@@
 <wire x1="69.6875" y1="4.375" x2="69.6875" y2="8.44" width="1.016" layer="1"/>
 <wire x1="69.6875" y1="8.44" x2="67.755" y2="10.3725" width="1.016" layer="1"/>
+<contactref element="R2" pad="1"/>
+<wire x1="67.8975" y1="13.135" x2="67.755" y2="12.9925" width="1.27" layer="1"/>
+<wire x1="67.755" y1="12.9925" x2="67.755" y2="10.3725" width="1.27" layer="1"/>
 </signal>
 <signal name="SCL">
@@
 <wire x1="65.3125" y1="9.0625" x2="65.3125" y2="10.275" width="1.27" layer="1"/>
 <wire x1="65.3125" y1="10.275" x2="65.215" y2="10.3725" width="1.27" layer="1"/>
+<contactref element="R3" pad="1"/>
+<wire x1="65.185" y1="13.175" x2="65.215" y2="13.145" width="1.27" layer="1"/>
+<wire x1="65.215" y1="13.145" x2="65.215" y2="10.3725" width="1.27" layer="1"/>
 </signal>
 <signal name="C">
@@
 <wire x1="35.625" y1="35" x2="35.625" y2="37.1875" width="1.27" layer="1"/>
 <wire x1="35.625" y1="37.1875" x2="42.5" y2="44.0625" width="1.27" layer="1"/>
-<wire x1="42.5" y1="44.0625" x2="55.05" y2="53.55" width="0" layer="19" extent="1-1"/>
+<wire x1="42.5" y1="44.0625" x2="49.6875" y2="44.0625" width="1.27" layer="1"/>
+<wire x1="49.6875" y1="44.0625" x2="55" y2="49.375" width="1.27" layer="1"/>
+<wire x1="55" y1="49.375" x2="55" y2="53.5" width="1.27" layer="1"/>
+<wire x1="55" y1="53.5" x2="55.05" y2="53.55" width="1.27" layer="1"/>
 </signal>
 <signal name="A">
