File: target/arduino_encoder_tester/hardware/arduino-shield.sch (EAGLE design)
At the start: 5 parts, among them SW1 EC12E_SW

Commit message: seq_blm update
Parts:
- added R2, R3: (no value), rcl:R-EU_R0805
Connections:
- net SCL: now also R3.1
- net SDA: now also R2.1
- net VCC: now also R2.2, R3.2
Changed lines of the file:
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@@
 <part name="SW1" library="switch-alps" deviceset="EC12E_SW" device=""/>
 <part name="R1" library="rcl" deviceset="R-EU_" device="R0805"/>
+<part name="R2" library="rcl" deviceset="R-EU_" device="R0805"/>
+<part name="R3" library="rcl" deviceset="R-EU_" device="R0805"/>
 </parts>
 <sheets>
@@
 <instance part="SW1" gate="G$2" x="210.82" y="119.38"/>
 <instance part="R1" gate="G$1" x="160.02" y="109.22"/>
+<instance part="R2" gate="G$1" x="160.02" y="134.62"/>
+<instance part="R3" gate="G$1" x="172.72" y="132.08"/>
 </instances>
 <busses>
@@
 <label x="167.64" y="109.22" size="1.778" layer="95"/>
 </segment>
+<segment>
+<pinref part="R2" gate="G$1" pin="2"/>
+<wire x1="165.1" y1="134.62" x2="167.64" y2="134.62" width="0.1524" layer="91"/>
+<label x="162.56" y="137.16" size="1.778" layer="95"/>
+</segment>
+<segment>
+<pinref part="R3" gate="G$1" pin="2"/>
+<wire x1="177.8" y1="132.08" x2="182.88" y2="132.08" width="0.1524" layer="91"/>
+<label x="177.8" y="137.16" size="1.778" layer="95"/>
+</segment>
 </net>
 <net name="LIGHT" class="0">
@@
 <wire x1="144.78" y1="134.62" x2="154.94" y2="134.62" width="0.1524" layer="91"/>
 <label x="147.32" y="134.62" size="1.778" layer="95"/>
+<pinref part="R2" gate="G$1" pin="1"/>
 </segment>
 <segment>
@@
 <segment>
 <pinref part="SV2" gate="1" pin="3"/>
-<wire x1="144.78" y1="132.08" x2="154.94" y2="132.08" width="0.1524" layer="91"/>
+<wire x1="144.78" y1="132.08" x2="167.64" y2="132.08" width="0.1524" layer="91"/>
 <label x="147.32" y="132.08" size="1.778" layer="95"/>
-</segment>
-</net>
+<pinref part="R3" gate="G$1" pin="1"/>
+</segment>
+</net>
