File: target/seq__blm/hardware/button-led-matrix-4x4.brd (EAGLE design)
At the start: 100 x 100 mm, 152 parts, among them IC1 ATMEGA48/88/168-AU, IC2 AMS1117-3.3, X1 CRYSTALS-NOGND-HC49

Commit message: button-led-matrix-4x4 board v1.2
Parts:
- added PAD110: WIREPADSMD1,27-254, wirepad:SMD1,27-2,54
Connections:
- new net N$11: PAD84.1
- net B7: now also PAD110.1
Routing:
- net B7: track 1.86 -> 7.01 mm
Other:
- board text added: "I2C ADDRESS:"
- board text added: "QC:"
- board text added: "v1.2"
- board text removed: "v1.1"
Changed lines of the file:
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@@
 <text x="31.875" y="71.875" size="1.016" layer="22" rot="MR0">CUT</text>
 <text x="55" y="95.625" size="2.54" layer="21" font="vector">16 LED+BUTTON PAD</text>
-<text x="88.125" y="1.875" size="2.54" layer="21">v1.1</text>
+<text x="34.375" y="96.25" size="2.54" layer="21">v1.2</text>
 <text x="20.625" y="55.625" size="1.016" layer="21" rot="R90">INT</text>
 <text x="21.875" y="55.625" size="1.016" layer="21" rot="R90">SDA</text>
@@
 <text x="15.9512" y="27.2288" size="1.778" layer="21">C</text>
 <text x="15.9512" y="2.2352" size="1.778" layer="21">D</text>
+<text x="96.875" y="57.5" size="1.778" layer="22" rot="MR0">SCK</text>
+<text x="97.5" y="60" size="1.778" layer="22" rot="MR0">MISO</text>
+<text x="5.625" y="96.875" size="1.778" layer="21">QC:</text>
+<wire x1="5" y1="99.375" x2="18.125" y2="99.375" width="0.4064" layer="21"/>
+<wire x1="18.125" y1="99.375" x2="18.125" y2="96.25" width="0.4064" layer="21"/>
+<wire x1="18.125" y1="96.25" x2="5" y2="96.25" width="0.4064" layer="21"/>
+<wire x1="5" y1="96.25" x2="5" y2="99.375" width="0.4064" layer="21"/>
+<wire x1="55" y1="0.625" x2="94.375" y2="0.625" width="0.4064" layer="21"/>
+<wire x1="94.375" y1="0.625" x2="94.375" y2="4.375" width="0.4064" layer="21"/>
+<wire x1="94.375" y1="4.375" x2="55" y2="4.375" width="0.4064" layer="21"/>
+<wire x1="55" y1="4.375" x2="55" y2="0.625" width="0.4064" layer="21"/>
+<text x="55.625" y="1.25" size="1.778" layer="21">I2C ADDRESS:</text>
 </plain>
 <attributes>
@@
 <element name="C18" library="rcl" package="C0805" value="0.1" x="62.5" y="37.5" rot="MR90"/>
 <element name="C19" library="rcl" package="C0805" value="0.1" x="87.5" y="37.5" rot="MR90"/>
+<element name="PAD110" library="wirepad" package="SMD1,27-2,54" value="WIREPADSMD1,27-254" x="60.625" y="65.625" rot="MR180"/>
 </elements>
 <signals>
@@
 <wire x1="54.449540625" y1="64.1211125" x2="55.588" y2="65.259571875" width="0.4064" layer="16"/>
 <wire x1="55.588" y1="65.259571875" x2="55.588" y2="65.513" width="0.4064" layer="16"/>
+<contactref element="PAD110" pad="1"/>
+<wire x1="60.625" y1="65.625" x2="55.588" y2="65.625" width="0.4064" layer="16"/>
+<wire x1="55.588" y1="65.625" x2="55.588" y2="65.513" width="0.4064" layer="16"/>
 </signal>
 <signal name="B8">
@@
 <via x="87.5" y="72.5" extent="1-16" drill="0.6" shape="octagon"/>
 </signal>
+<signal name="N$11">
+<contactref element="PAD84" pad="1"/>
+</signal>
 </signals>
