File: target/seq__blm/hardware/button-led-matrix-4x4.sch (EAGLE design)
At the start: 152 parts, among them IC1 ATMEGA48/88/168-AU, IC2 AMS1117-3.3, X1 CRYSTALS-NOGND-HC49

Commit message: button-led-matrix-4x4 board v1.2
Parts:
- added PAD110: WIREPADSMD1,27-254, wirepad:WIREPADSMD1,27-254
Connections:
- new net N$11: PAD84.P
- net B7: now also PAD110.P
Changed lines of the file:
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@@
 <part name="C18" library="rcl" deviceset="C-EU" device="C0805" value="0.1"/>
 <part name="C19" library="rcl" deviceset="C-EU" device="C0805" value="0.1"/>
+<part name="PAD110" library="wirepad" deviceset="WIREPAD" device="SMD1,27-254"/>
 </parts>
 <sheets>
@@
 <instance part="C18" gate="G$1" x="73.66" y="-149.86"/>
 <instance part="C19" gate="G$1" x="66.04" y="-149.86"/>
+<instance part="PAD110" gate="G$1" x="162.56" y="-137.16"/>
 </instances>
 <busses>
@@
 <label x="162.56" y="-73.66" size="1.778" layer="95"/>
 </segment>
+<segment>
+<pinref part="PAD110" gate="G$1" pin="P"/>
+<wire x1="165.1" y1="-137.16" x2="187.96" y2="-137.16" width="0.1524" layer="91"/>
+<label x="180.34" y="-137.16" size="1.778" layer="95"/>
+</segment>
 </net>
 <net name="B8" class="0">
@@
 </segment>
 </net>
+<net name="N$11" class="0">
+<segment>
+<pinref part="PAD84" gate="G$1" pin="P"/>
+<wire x1="165.1" y1="-129.54" x2="187.96" y2="-129.54" width="0.1524" layer="91"/>
+</segment>
+</net>
