File: target/split-keyboard-dongle/hardware/SplitKbHub.kicad_pcb (KiCad board)
At the start: 2 copper layers, 200 x 200 mm, 8 parts, among them U2 YAAJ_BluePill_Part_Like, U3 TRRS, U5 TRRS, U6 TRRS

Commit message: SplitKbHub.kicad_pcb
Other:
- board size 200 x 200 mm -> 23.7 x 66.4 mm
