File: target/just-split/hardware/just-split.kicad_pcb (KiCad board)
At the start: 2 copper layers, 128.2 x 112.4 mm, 122 parts, among them J1 MJ-4PP-9, J2 OLED, J3 MJ-4PP-9, Q1 MMBT3904, Q2 MMBT3904, Q3 MMBT3904, Q4 MMBT3904, SW1 SW_PUSH, SW10 SW_PUSH, SW11 SW_PUSH, SW12 SW_PUSH, SW14 SW_PUSH, SW15 SW_PUSH, SW16 SW_PUSH, SW17 SW_PUSH, SW18 SW_PUSH, SW19 SW_PUSH, SW2 SW_PUSH, SW20 SW_PUSH, SW3 SW_PUSH, SW4 SW_PUSH, SW5 SW_PUSH, SW6 SW_PUSH, SW7 SW_PUSH, SW8 SW_PUSH, SW9 SW_PUSH, U1 ATmega88-20PU, U2 ATmega88-20PU

Commit message: just-split hw update (v0.2)
Parts:
- added C4: 0.1, Capacitor_SMD:C_0805_2012Metric_Pad1.18x1.45mm_HandSolder, F.Cu at (84.2, 95.1)
- added C5: 0.1, Capacitor_SMD:C_0805_2012Metric_Pad1.18x1.45mm_HandSolder, B.Cu at (97.5, 95.2)
- added R25: 10k, Resistor_SMD:R_0805_2012Metric_Pad1.20x1.40mm_HandSolder, B.Cu at (202.0, 78.7)
- added R26: 10k, Resistor_SMD:R_0805_2012Metric_Pad1.20x1.40mm_HandSolder, B.Cu at (197.5, 78.7)
- added R27: 10k, Resistor_SMD:R_0805_2012Metric_Pad1.20x1.40mm_HandSolder, B.Cu at (191.2, 78.9)
- added R28: 10k, Resistor_SMD:R_0805_2012Metric_Pad1.20x1.40mm_HandSolder, B.Cu at (187.0, 78.9)
- moved R18 22.6 mm to (187.7, 129.6), turned to 180 degrees
- moved JP2 0.40 mm to (188.2, 87.2)
- moved JP3 0.40 mm to (185.7, 87.2)
- moved JP4 0.40 mm to (183.2, 87.2)
- moved JP5 0.40 mm to (180.7, 87.2)
- moved JP6 0.40 mm to (188.2, 87.2)
- moved JP7 0.40 mm to (185.7, 87.2)
- moved JP8 0.40 mm to (183.2, 87.2)
- moved JP9 0.40 mm to (180.7, 87.2)
Routing:
- net VCC: track 865.7 -> 889.6 mm
- net SCL: track 69.0 -> 77.6 mm
- net /RESET: track 65.9 -> 70.6 mm
- net row0: track 237.8 -> 242.2 mm
- net row3: track 197.2 -> 201.6 mm, vias 5 -> 6
- net row2: track 228.1 -> 231.8 mm, vias 13 -> 14
- net Net-(L18-Pad3): track 31.6 -> 34.7 mm, vias 3 -> 4
- net GND: track 870.3 -> 873.3 mm, vias 42 -> 43
- net col5: track 194.0 -> 196.2 mm
- net row1: track 233.8 -> 235.3 mm, vias 11 -> 12
- net SDA: track 70.4 -> 71.6 mm
- net (no net): vias 13 -> 11
Other:
- board text added: "* Q1..Q4 should have had pull-up resistors"
- board text added: "* R21(?) had a short with VCC(GND?) - cut"
- board text added: "* pin 1 of L20 unconnected"
- board text added: "Errata for v0.1:"
- board text added: "v0.2"
- board text removed: "v0.1"
