File: target/just-split/hardware/just-split.sch (KiCad schematic (older format))
At the start: 122 parts, among them J1 MJ-4PP-9, J2 OLED, J3 MJ-4PP-9, Q1 MMBT3904, Q2 MMBT3904, Q3 MMBT3904, Q4 MMBT3904, SW1 SW_PUSH, SW10 SW_PUSH, SW11 SW_PUSH, SW12 SW_PUSH, SW14 SW_PUSH, SW15 SW_PUSH, SW16 SW_PUSH, SW17 SW_PUSH, SW18 SW_PUSH, SW19 SW_PUSH, SW2 SW_PUSH, SW20 SW_PUSH, SW3 SW_PUSH, SW4 SW_PUSH, SW5 SW_PUSH, SW6 SW_PUSH, SW7 SW_PUSH, SW8 SW_PUSH, SW9 SW_PUSH, U1 ATmega88-20PU, U2 ATmega88-20PU

Commit message: just-split hw update (v0.2)
Parts:
- added C4, C5: 0.1, Capacitor_SMD:C_0805_2012Metric_Pad1.18x1.45mm_HandSolder, symbol Device:C
- added R25, R26, R27, R28: 10k, Resistor_SMD:R_0805_2012Metric_Pad1.20x1.40mm_HandSolder, symbol Device:R
Connections:
- wire segments 388 -> 398
Other:
- note added: "(RECOMMENDED)"
- note added: "ROW PULL-UPS"
- moved on the sheet: C1, C2, C3, J1, J3, Q1, Q2, Q3, Q4, R10, R11, R12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
