File: target/future-kb/hardware/just-split.kicad_pcb (KiCad board)
At the start: 2 copper layers, 67 parts, among them J1 MJ-4PP-9, U1 ATmega88-20PU

Commit message: future-kb: kicad_pcb
Parts:
- moved TP35 15.4 mm to (71.5, 145.4), turned to 90 degrees
- moved TP33 13.5 mm to (68.9, 145.4), turned to 90 degrees
- moved TP25 12.8 mm to (71.5, 142.9), turned to 90 degrees
- moved TP31 12.4 mm to (66.2, 145.4), turned to 90 degrees
- moved TP15 10.6 mm to (71.5, 140.3), turned to 90 degrees
- moved TP23 10.3 mm to (68.9, 142.9), turned to 90 degrees
- moved TP5 9.43 mm to (71.5, 137.8), turned to 90 degrees
- moved TP1 8.88 mm to (66.2, 142.9), turned to 90 degrees
- moved D11 8.21 mm to (40.4, 129.9)
- moved D12 8.21 mm to (40.4, 139.0)
- moved D13 8.21 mm to (40.4, 143.5)
- moved D14 8.21 mm to (40.4, 134.4)
- moved D15 8.21 mm to (40.4, 148.0)
- moved TP22 8.21 mm to (39.4, 132.0)
- moved TP24 8.21 mm to (39.4, 141.0)
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Routing:
- net /VCC: track 76.8 -> 42.4 mm
- net SDA: track 35.6 -> 26.1 mm
- net col3: track 12.6 -> 20.7 mm
- net col2: track 14.3 -> 20.5 mm
- net row3: track 22.7 -> 27.1 mm
- net row2: track 29.9 -> 33.7 mm
- net GND: track 70.0 -> 67.8 mm
- net col1: track 14.5 -> 16.4 mm
- net SCL: track 15.2 -> 16.5 mm
Other:
- board outline added: 38 x 52.5 mm
