File: target/future-kb/hardware/wireless-v1/just-split.kicad_sch (KiCad schematic)
At the start: 4 parts, among them J1 Conn_02x12_Odd_Even, J6 Conn_02x12_Odd_Even, J7 Conn_02x10_Odd_Even, U1 HOLYIOT-18010-NRF52840_Simple

Commit message: future-kb: fixes
Parts:
- added C1: C, Capacitor_SMD:C_0805_2012Metric, symbol Device:C
Connections:
- net GND: now also C1.2
Changed lines of the file:
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@@
+    (stroke (width 0) (type default) (color 0 0 0 0))
+  )
+  (wire (pts (xy 53.34 107.95) (xy 53.34 116.84))
     (stroke (width 0) (type default) (color 0 0 0 0))
   )
@@
     (stroke (width 0) (type default) (color 0 0 0 0))
   )
+  (wire (pts (xy 53.34 124.46) (xy 53.34 133.35))
+    (stroke (width 0) (type default) (color 0 0 0 0))
+  )
   (wire (pts (xy 151.13 109.22) (xy 165.1 109.22))
     (stroke (width 0) (type default) (color 0 0 0 0))
@@
   )
   (label "P23" (at 266.7 115.57 0)
+    (effects (font (size 1.27 1.27)) (justify left bottom))
+  )
+  (label "GND" (at 53.34 133.35 0)
     (effects (font (size 1.27 1.27)) (justify left bottom))
   )
@@
     (pin "9")
   )
+  (symbol (lib_id "Device:C") (at 53.34 120.65 0) (unit 1)
+    (in_bom yes) (on_board yes) (fields_autoplaced)
+    (property "Reference" "C1" (id 0) (at 57.15 119.3799 0)
+      (effects (font (size 1.27 1.27)) (justify left))
+    )
+    (property "Value" "C" (id 1) (at 57.15 121.9199 0)
+      (effects (font (size 1.27 1.27)) (justify left))
+    )
+    (property "Footprint" "Capacitor_SMD:C_0805_2012Metric" (id 2) (at 54.3052 124.46 0)
+      (effects (font (size 1.27 1.27)) hide)
+    )
+    (property "Datasheet" "~" (id 3) (at 53.34 120.65 0)
+      (effects (font (size 1.27 1.27)) hide)
+    )
+    (pin "1")
+    (pin "2")
+  )
   (sheet_instances
     (path "/" (page "1"))
   )
   (symbol_instances
+    (path "/e714757f-d7f7-427c-98e8-d6b2d76dfe81"
+      (reference "C1") (unit 1) (value "C") (footprint "Capacitor_SMD:C_0805_2012Metric")
+    )
     (path "/3078da7f-2d3b-4153-8bef-a90a1be562f7"
       (reference "J1") (unit 1) (value "Conn_02x12_Odd_Even") (footprint "Connector_PinHeader_2.54mm:PinHeader_2x12_P2.54mm_Vertical")
