File: target/plc-4u-a/hardware/plc-4u-a/top_board.kicad_sch (KiCad schematic)
At the start: 37 parts, among them J12 S3 S5 LEDs, J23 S3 S5 LEDs, J24 S4 S6 LEDs, J27 S3BTN, J28 S4BTN, J29 S5BTN, J30 S6BTN, J40 Leak sensors, J41 TA_C, J42 TB_C, J43 TC_C, J44 TD_C, J48 S3 S5 LEDs

Commit message: update
Parts:
- added J67: VDD VSS, Connector_PinHeader_2.54mm:PinHeader_1x02_P2.54mm_Vertical, symbol Connector:Conn_01x02_Male
- added J75, J76: VSS, Connector_PinHeader_2.54mm:PinHeader_1x01_P2.54mm_Vertical, symbol Connector:Conn_01x01_Male
- added J78: VDD, Connector_PinHeader_2.54mm:PinHeader_1x01_P2.54mm_Vertical, symbol Connector:Conn_01x01_Male
Connections:
- net VDD: now also J67.2 (Pin_2), J78.1 (Pin_1)
- net VSS: now also J67.1 (Pin_1), J75.1 (Pin_1), J76.1 (Pin_1)
Changed lines of the file:
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@@
+    (stroke (width 0) (type default) (color 0 0 0 0))
+  )
+  (wire (pts (xy 81.28 167.64) (xy 86.36 167.64))
     (stroke (width 0) (type default) (color 0 0 0 0))
   )
@@
     (stroke (width 0) (type default) (color 0 0 0 0))
   )
+  (wire (pts (xy 144.78 190.5) (xy 149.86 190.5))
+    (stroke (width 0) (type default) (color 0 0 0 0))
+  )
   (wire (pts (xy 30.48 162.56) (xy 40.64 162.56))
     (stroke (width 0) (type default) (color 0 0 0 0))
@@
     (stroke (width 0) (type default) (color 0 0 0 0))
   )
+  (wire (pts (xy 81.28 170.18) (xy 86.36 170.18))
+    (stroke (width 0) (type default) (color 0 0 0 0))
+  )
   (wire (pts (xy 149.86 124.46) (xy 170.18 124.46))
     (stroke (width 0) (type default) (color 0 0 0 0))
@@
     (stroke (width 0) (type default) (color 0 0 0 0))
   )
+  (wire (pts (xy 157.48 190.5) (xy 162.56 190.5))
+    (stroke (width 0) (type default) (color 0 0 0 0))
+  )
   (wire (pts (xy 236.22 35.56) (xy 238.76 35.56))
     (stroke (width 0) (type default) (color 0 0 0 0))
@@
     (stroke (width 0) (type default) (color 0 0 0 0))
   )
+  (wire (pts (xy 132.08 190.5) (xy 137.16 190.5))
+    (stroke (width 0) (type default) (color 0 0 0 0))
+  )
   (wire (pts (xy 236.22 40.64) (xy 238.76 40.64))
     (stroke (width 0) (type default) (color 0 0 0 0))
@@
     (effects (font (size 1.27 1.27)) (justify left bottom))
   )
+  (label "VSS" (at 132.715 190.5 0)
+    (effects (font (size 1.27 1.27)) (justify left bottom))
+  )
   (label "VSS" (at 241.3 129.54 0)
     (effects (font (size 1.27 1.27)) (justify left bottom))
   )
+  (label "VDD" (at 81.915 170.18 0)
+    (effects (font (size 1.27 1.27)) (justify left bottom))
+  )
   (label "S5BTN" (at 190.5 124.46 0)
     (effects (font (size 1.27 1.27)) (justify left bottom))
@@
     (effects (font (size 1.27 1.27)) (justify left bottom))
   )
+  (label "VDD" (at 158.115 190.5 0)
+    (effects (font (size 1.27 1.27)) (justify left bottom))
+  )
   (label "S1LED" (at 50.8 170.18 0)
     (effects (font (size 1.27 1.27)) (justify left bottom))
@@
     (effects (font (size 1.27 1.27)) (justify left bottom))
   )
+  (label "VSS" (at 81.915 167.64 0)
+    (effects (font (size 1.27 1.27)) (justify left bottom))
+  )
   (label "S1LED" (at 50.8 129.54 0)
+    (effects (font (size 1.27 1.27)) (justify left bottom))
+  )
+  (label "VSS" (at 145.415 190.5 0)
     (effects (font (size 1.27 1.27)) (justify left bottom))
   )
@@
     (pin "4")
   )
+  (symbol (lib_id "Connector:Conn_01x01_Male") (at 152.4 190.5 0) (unit 1)
+    (in_bom yes) (on_board yes)
+    (property "Reference" "J78" (id 0) (at 153.67 177.8 0))
+    (property "Value" "VDD" (id 1) (at 154.94 180.34 0))
+    (property "Footprint" "Connector_PinHeader_2.54mm:PinHeader_1x01_P2.54mm_Vertical" (id 2) (at 152.4 190.5 0)
+      (effects (font (size 1.27 1.27)) hide)
+    )
+    (property "Datasheet" "~" (id 3) (at 152.4 190.5 0)
+      (effects (font (size 1.27 1.27)) hide)
+    )
+    (pin "1")
+  )
   (symbol (lib_id "Device:R") (at 242.57 35.56 90) (unit 1)
     (in_bom yes) (on_board yes)
@@
     (pin "1")
   )
+  (symbol (lib_id "Connector:Conn_01x01_Male") (at 139.7 190.5 0) (unit 1)
+    (in_bom yes) (on_board yes)
+    (property "Reference" "J76" (id 0) (at 140.97 177.8 0))
+    (property "Value" "VSS" (id 1) (at 142.24 180.34 0))
+    (property "Footprint" "Connector_PinHeader_2.54mm:PinHeader_1x01_P2.54mm_Vertical" (id 2) (at 139.7 190.5 0)
+      (effects (font (size 1.27 1.27)) hide)
+    )
+    (property "Datasheet" "~" (id 3) (at 139.7 190.5 0)
+      (effects (font (size 1.27 1.27)) hide)
+    )
+    (pin "1")
+  )
   (symbol (lib_id "Connector:Conn_01x01_Male") (at 251.46 35.56 180) (unit 1)
     (in_bom yes) (on_board yes)
@@
     (pin "1")
     (pin "2")
+  )
+  (symbol (lib_id "Connector:Conn_01x01_Male") (at 127 190.5 0) (unit 1)
+    (in_bom yes) (on_board yes)
+    (property "Reference" "J75" (id 0) (at 128.27 177.8 0))
+    (property "Value" "VSS" (id 1) (at 129.54 180.34 0))
+    (property "Footprint" "Connector_PinHeader_2.54mm:PinHeader_1x01_P2.54mm_Vertical" (id 2) (at 127 190.5 0)
+      (effects (font (size 1.27 1.27)) hide)
+    )
+    (property "Datasheet" "~" (id 3) (at 127 190.5 0)
+      (effects (font (size 1.27 1.27)) hide)
+    )
+    (pin "1")
   )
   (symbol (lib_id "Device:R") (at 191.77 35.56 90) (unit 1)
@@
     (pin "3")
   )
+  (symbol (lib_id "Connector:Conn_01x02_Male") (at 76.2 167.64 0) (unit 1)
+    (in_bom yes) (on_board yes)
+    (property "Reference" "J67" (id 0) (at 77.47 157.48 0))
+    (property "Value" "VDD VSS" (id 1) (at 81.28 160.02 0))
+    (property "Footprint" "Connector_PinHeader_2.54mm:PinHeader_1x02_P2.54mm_Vertical" (id 2) (at 76.2 167.64 0)
+      (effects (font (size 1.27 1.27)) hide)
+    )
+    (property "Datasheet" "~" (id 3) (at 76.2 167.64 0)
+      (effects (font (size 1.27 1.27)) hide)
+    )
+    (pin "1")
+    (pin "2")
+  )
   (symbol (lib_id "Device:R") (at 166.37 78.74 90) (unit 1)
