File: target/plc-4u-a/hardware/plc-4u-a/plc-4u-a.kicad_pcb (KiCad board)
At the start: 2 copper layers, 64 x 84 mm, 41 parts, among them J1 Screw_Terminal_01x02, J10 Screw_Terminal_01x02, J11 Conn_01x04_Male, J12 Conn_01x04_Male, J2 Screw_Terminal_01x02, J3 Screw_Terminal_01x02, J4 Screw_Terminal_01x02, J5 Screw_Terminal_01x02, J6 Screw_Terminal_01x02, J7 Screw_Terminal_01x02, J8 Screw_Terminal_01x02, J9 Screw_Terminal_01x02, Q1 IRF4905, Q2 IRF4905, Q3 IRF4905, Q4 IRF4905, U1 ATmega16-16P, U2 PC817, U3 PC817, U4 PC817, U5 PC817, Y1 Crystal

Commit message: update
Parts:
- added D1: FR157, Diode_THT:D_DO-41_SOD81_P10.16mm_Horizontal, F.Cu at (63.7, 135.6)
- added D1: LED_Dual_KAK, LED_THT:LED_Rectangular_W5.0mm_H2.0mm-3Pins, F.Cu at (373.9, 85.0)
- added D2: LED_Dual_KAK, LED_THT:LED_Rectangular_W5.0mm_H2.0mm-3Pins, F.Cu at (388.9, 85.0)
- added D3: LED_Dual_KAK, LED_THT:LED_Rectangular_W5.0mm_H2.0mm-3Pins, F.Cu at (406.0, 85.0)
- added D4: LED_Dual_KAK, LED_THT:LED_Rectangular_W5.0mm_H2.0mm-3Pins, F.Cu at (420.9, 85.0)
- added J13: Valve control in, Connector_PinHeader_2.54mm:PinHeader_1x04_P2.54mm_Vertical, F.Cu at (103.9, 85.8)
- added J14: Leak sensors, Connector_PinHeader_2.54mm:PinHeader_1x04_P2.54mm_Vertical, F.Cu at (86.1, 85.8)
- added J15: I2C, Connector_PinHeader_2.54mm:PinHeader_1x02_P2.54mm_Vertical, F.Cu at (121.6, 85.8)
- added J16: I2C, Connector_PinHeader_2.54mm:PinHeader_1x02_P2.54mm_Vertical, F.Cu at (221.6, 85.8)
- added J17: Display, Connector_PinHeader_2.54mm:PinHeader_1x04_P2.54mm_Vertical, F.Cu at (169.9, 98.3)
- added J18: X leds btns, Connector_PinHeader_2.54mm:PinHeader_1x04_P2.54mm_Vertical, F.Cu at (193.7, 106.0)
- added J19: Valve leds, Connector_PinHeader_2.54mm:PinHeader_1x04_P2.54mm_Vertical, F.Cu at (114.0, 106.0)
- added J20: Valve leds, Connector_PinHeader_2.54mm:PinHeader_1x04_P2.54mm_Vertical, F.Cu at (214.0, 106.0)
- added J21: Leak sensors, Connector_PinHeader_2.54mm:PinHeader_1x04_P2.54mm_Vertical, F.Cu at (186.1, 85.8)
- added J22: Valve control in, Connector_PinHeader_2.54mm:PinHeader_1x04_P2.54mm_Vertical, F.Cu at (203.9, 85.8)
- added J23: S3 S5 LEDs, Connector_PinHeader_2.54mm:PinHeader_1x02_P2.54mm_Vertical, F.Cu at (401.5, 101.2)
- added J24: S4 S6 LEDs, Connector_PinHeader_2.54mm:PinHeader_1x02_P2.54mm_Vertical, F.Cu at (430.2, 101.2)
- added J25: S3 S5 LEDs, Connector_PinHeader_2.54mm:PinHeader_1x02_P2.54mm_Vertical, F.Cu at (201.5, 101.2)
- added J26: S4 S6 LEDs, Connector_PinHeader_2.54mm:PinHeader_1x02_P2.54mm_Vertical, F.Cu at (230.2, 101.2)
- added J27: S3BTN, Connector_PinHeader_2.54mm:PinHeader_1x01_P2.54mm_Vertical, F.Cu at (401.3, 87.7)
- added J28: S4BTN, Connector_PinHeader_2.54mm:PinHeader_1x01_P2.54mm_Vertical, F.Cu at (430.2, 87.7)
- added J29: S5BTN, Connector_PinHeader_2.54mm:PinHeader_1x01_P2.54mm_Vertical, F.Cu at (401.3, 117.2)
- added J30: S6BTN, Connector_PinHeader_2.54mm:PinHeader_1x01_P2.54mm_Vertical, F.Cu at (430.2, 117.2)
- added J31: S3BTN, Connector_PinHeader_2.54mm:PinHeader_1x01_P2.54mm_Vertical, F.Cu at (201.3, 87.7)
- added J32: S4BTN, Connector_PinHeader_2.54mm:PinHeader_1x01_P2.54mm_Vertical, F.Cu at (230.2, 87.7)
- added J33: S5BTN, Connector_PinHeader_2.54mm:PinHeader_1x01_P2.54mm_Vertical, F.Cu at (201.3, 117.2)
- added J34: S6BTN, Connector_PinHeader_2.54mm:PinHeader_1x01_P2.54mm_Vertical, F.Cu at (230.2, 117.2)
- added J35: PWR_OUT, TerminalBlock_Phoenix:TerminalBlock_Phoenix_MKDS-1,5-2-5.08_1x02_P5.08mm_Horizontal, F.Cu at (182.2, 72.2)
- added J36: Sensors AB, TerminalBlock_Phoenix:TerminalBlock_Phoenix_MKDS-1,5-2-5.08_1x02_P5.08mm_Horizontal, F.Cu at (197.4, 72.2)
- added J37: Sensors CD, TerminalBlock_Phoenix:TerminalBlock_Phoenix_MKDS-1,5-2-5.08_1x02_P5.08mm_Horizontal, F.Cu at (207.6, 72.2)
- added J38: PWR_OUT, TerminalBlock_Phoenix:TerminalBlock_Phoenix_MKDS-1,5-2-5.08_1x02_P5.08mm_Horizontal, F.Cu at (222.8, 72.2)
- added R13: 820, Resistor_SMD:R_0805_2012Metric, B.Cu at (98.0, 81.8)
- added R14: 820, Resistor_SMD:R_0805_2012Metric, B.Cu at (82.4, 82.8)
- added R15: 820, Resistor_SMD:R_0805_2012Metric, B.Cu at (78.4, 84.4)
- added R16: 820, Resistor_SMD:R_0805_2012Metric, B.Cu at (63.4, 90.1)
- added R17: R, Resistor_THT:R_Axial_DIN0207_L6.3mm_D2.5mm_P10.16mm_Horizontal, F.Cu at (201.5, 98.7)
- added R18: R, Resistor_THT:R_Axial_DIN0207_L6.3mm_D2.5mm_P10.16mm_Horizontal, F.Cu at (230.2, 98.7)
- added R19: R, Resistor_THT:R_Axial_DIN0207_L6.3mm_D2.5mm_P10.16mm_Horizontal, F.Cu at (201.5, 108.8)
- added R20: R, Resistor_THT:R_Axial_DIN0207_L6.3mm_D2.5mm_P10.16mm_Horizontal, F.Cu at (230.2, 108.8)
- added R21: R, Resistor_SMD:R_1206_3216Metric, B.Cu at (109.0, 66.5)
- added R22: R, Resistor_SMD:R_1206_3216Metric, B.Cu at (103.3, 66.5)
- added R23: R, Resistor_SMD:R_1206_3216Metric, B.Cu at (97.5, 66.5)
- added R24: R, Resistor_SMD:R_1206_3216Metric, B.Cu at (91.4, 66.5)
- added R25: R, Resistor_SMD:R_1206_3216Metric, B.Cu at (87.3, 66.5)
- added R26: R, Resistor_SMD:R_1206_3216Metric, B.Cu at (82.2, 66.5)
- added R27: R, Resistor_SMD:R_1206_3216Metric, B.Cu at (121.8, 126.6)
- added R28: R, Resistor_SMD:R_1206_3216Metric, B.Cu at (127.8, 114.2)
- added R29: R, Resistor_SMD:R_1206_3216Metric, B.Cu at (144.2, 84.3)
- added R30: R, Resistor_SMD:R_1206_3216Metric, B.Cu at (120.7, 66.5)
- added R31: R, Resistor_SMD:R_1206_3216Metric, B.Cu at (114.7, 66.5)
- added S1: MOMENTARY-SWITCH-SPST-LED-PTH-12MM, mod:TACTILE_SWITCH_LED_PTH_12MM, F.Cu at (376.5, 110.5)
- added S2: MOMENTARY-SWITCH-SPST-LED-PTH-12MM, mod:TACTILE_SWITCH_LED_PTH_12MM, F.Cu at (391.5, 110.5)
- added S3: MOMENTARY-SWITCH-SPST-LED-PTH-12MM, mod:TACTILE_SWITCH_LED_PTH_12MM, F.Cu at (408.5, 94.5)
- added S4: MOMENTARY-SWITCH-SPST-LED-PTH-12MM, mod:TACTILE_SWITCH_LED_PTH_12MM, F.Cu at (423.5, 94.5)
- added S5: MOMENTARY-SWITCH-SPST-LED-PTH-12MM, mod:TACTILE_SWITCH_LED_PTH_12MM, F.Cu at (408.5, 110.5)
- added S6: MOMENTARY-SWITCH-SPST-LED-PTH-12MM, mod:TACTILE_SWITCH_LED_PTH_12MM, F.Cu at (423.5, 110.5)
- added U10: PC817, Package_DIP:DIP-4_W7.62mm, F.Cu at (117.3, 70.2)
- added U11: PC817, Package_DIP:DIP-4_W7.62mm, F.Cu at (111.5, 70.2)
- added U12: PC817, Package_DIP:DIP-4_W7.62mm, F.Cu at (105.8, 70.2)
- added U13: PC817, Package_DIP:DIP-4_W7.62mm, F.Cu at (100.1, 70.2)
- added U14: PC817, Package_DIP:DIP-4_W7.62mm, F.Cu at (94.0, 70.2)
- added U15: PC817, Package_DIP:DIP-4_W7.62mm, F.Cu at (81.1, 72.2)
- added U16: PC817, Package_DIP:DIP-4_W7.62mm, F.Cu at (75.5, 72.2)
- added U17: PC817, Package_DIP:DIP-4_W7.62mm, F.Cu at (57.5, 68.5)
- added U6: PC817, Package_DIP:DIP-4_W7.62mm, F.Cu at (110.7, 118.3)
- added U7: PC817, Package_DIP:DIP-4_W7.62mm, F.Cu at (116.2, 118.3)
- added U8: PC817, Package_DIP:DIP-4_W7.62mm, F.Cu at (130.4, 84.4)
- added U9: PC817, Package_DIP:DIP-4_W7.62mm, F.Cu at (123.2, 70.2)
- J1, J2, J3, J4, J5: footprint TerminalBlock_Phoenix:TerminalBlock_Phoenix_MKDS-1,5-2_1x02_P5.00mm_Horizontal -> TerminalBlock_Phoenix:TerminalBlock_Phoenix_MKDS-1,5-2-5.08_1x02_P5.08mm_Horizontal
- J10: value Screw_Terminal_01x02 -> X_INS; footprint TerminalBlock_Phoenix:TerminalBlock_Phoenix_MKDS-1,5-2_1x02_P5.00mm_Horizontal -> TerminalBlock_Phoenix:TerminalBlock_Phoenix_MKDS-1,5-2-5.08_1x02_P5.08mm_Horizontal
- J11: value Conn_01x04_Male -> X Leds Btns
- J12: value Conn_01x04_Male -> Display
- J6: value Screw_Terminal_01x02 -> V_ST_HWS; footprint TerminalBlock_Phoenix:TerminalBlock_Phoenix_MKDS-1,5-2_1x02_P5.00mm_Horizontal -> TerminalBlock_Phoenix:TerminalBlock_Phoenix_MKDS-1,5-2-5.08_1x02_P5.08mm_Horizontal
- J7: value Screw_Terminal_01x02 -> V_ST_CWS; footprint TerminalBlock_Phoenix:TerminalBlock_Phoenix_MKDS-1,5-2_1x02_P5.00mm_Horizontal -> TerminalBlock_Phoenix:TerminalBlock_Phoenix_MKDS-1,5-2-5.08_1x02_P5.08mm_Horizontal
- J8: value Screw_Terminal_01x02 -> W_CT_HWS; footprint TerminalBlock_Phoenix:TerminalBlock_Phoenix_MKDS-1,5-2_1x02_P5.00mm_Horizontal -> TerminalBlock_Phoenix:TerminalBlock_Phoenix_MKDS-1,5-2-5.08_1x02_P5.08mm_Horizontal
- J9: value Screw_Terminal_01x02 -> W_CT_CWS; footprint TerminalBlock_Phoenix:TerminalBlock_Phoenix_MKDS-1,5-2_1x02_P5.00mm_Horizontal -> TerminalBlock_Phoenix:TerminalBlock_Phoenix_MKDS-1,5-2-5.08_1x02_P5.08mm_Horizontal
- moved J12 261.1 mm to (369.9, 98.3), turned to 180 degrees
- moved H5 200.0 mm to (-128.5, 100.0)
- moved H6 100.0 mm to (0.00, 83.0)
- moved H7 100.0 mm to (28.5, 100.0)
- moved R12 2.54 mm to (100.0, 129.0)
- moved R2 2.54 mm to (79.0, 129.1)
- moved R6 2.54 mm to (86.0, 129.0)
- moved R9 2.54 mm to (93.0, 129.0)
- moved Y1 2.06 mm to (100.5, 109.5)
- moved R1 1.50 mm to (79.0, 124.0)
- moved R11 1.50 mm to (100.0, 124.0)
- moved R5 1.50 mm to (86.0, 124.0)
- moved R8 1.50 mm to (93.0, 124.0)
- moved J1 0.32 mm to (77.2, 138.0)
- moved J10 0.32 mm to (122.8, 62.0)
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Connections:
- J10 pad 1: unconnected-(J10-Pad1) -> /X9
- J10 pad 2: unconnected-(J10-Pad2) -> /X8
- J12 pad 1: /PD0 -> /Top board/GND
- J12 pad 2: /PD1 -> /Top board/VCC
- J12 pad 3: /PD2 -> /Top board/SCL
- J12 pad 4: /PD3 -> /Top board/SDA
- J6 pad 1: unconnected-(J6-Pad1) -> /X1
- J6 pad 2: unconnected-(J6-Pad2) -> /X0
- J7 pad 1: unconnected-(J7-Pad1) -> /X3
- J7 pad 2: unconnected-(J7-Pad2) -> /X2
- J8 pad 1: unconnected-(J8-Pad1) -> /X5
- J8 pad 2: unconnected-(J8-Pad2) -> /X4
- J9 pad 1: unconnected-(J9-Pad1) -> /X7
- J9 pad 2: unconnected-(J9-Pad2) -> /X6
- U1 pad 22: unconnected-(U1-Pad22) -> /SCL
- U1 pad 23: unconnected-(U1-Pad23) -> /SDA
- U1 pad 26: unconnected-(U1-Pad26) -> /PC4
- U1 pad 27: unconnected-(U1-Pad27) -> /PC5
- U1 pad 28: unconnected-(U1-Pad28) -> /PC6
- U1 pad 29: unconnected-(U1-Pad29) -> /PC7
- U1 pad 33: unconnected-(U1-Pad33) -> /PA7
- U1 pad 34: unconnected-(U1-Pad34) -> /PA6
- U1 pad 35: unconnected-(U1-Pad35) -> /PA5
- U1 pad 36: unconnected-(U1-Pad36) -> /PA4
- U1 pad 37: unconnected-(U1-Pad37) -> /PA3
- U1 pad 38: unconnected-(U1-Pad38) -> /PA2
- U1 pad 39: unconnected-(U1-Pad39) -> /PA1
- U1 pad 40: unconnected-(U1-Pad40) -> /PA0
Routing:
- net /Top board/GND: track 0.00 -> 100.8 mm
- net /VCC: track 55.8 -> 136.9 mm, vias 6 -> 7
- net /VSS: track 0.00 -> 63.9 mm
- net /Middle board/PC5: track 0.00 -> 46.6 mm
- net /Middle board/PC6: track 0.00 -> 34.0 mm
- net /Middle board/PC4: track 0.00 -> 20.0 mm
- net /Top board/S3BTN: track 0.00 -> 17.4 mm
- net /Top board/S5BTN: track 0.00 -> 17.4 mm
- net /Top board/S4BTN: track 0.00 -> 16.9 mm
- net /Top board/S6BTN: track 0.00 -> 16.9 mm
- net Net-(U16-Pad2): track 0.00 -> 11.6 mm
- net /PA3: track 0.00 -> 11.3 mm
- net Net-(U15-Pad2): track 0.00 -> 11.2 mm
- net /Middle board/PD4: track 0.00 -> 8.80 mm
- net /Middle board/PD3: track 0.00 -> 8.69 mm
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Other:
- board size 64 x 84 mm -> 363.5 x 84 mm

Commit message: update
Parts:
- removed the D1 at (63.7, 135.6)
- added D10: D, Diode_THT:D_DO-41_SOD81_P10.16mm_Horizontal, F.Cu at (126.1, 131.4)
- added D5: D, Diode_THT:D_DO-41_SOD81_P10.16mm_Horizontal, F.Cu at (76.5, 131.4)
- added D6: D, Diode_THT:D_DO-41_SOD81_P10.16mm_Horizontal, F.Cu at (84.4, 131.4)
- added D7: D, Diode_THT:D_DO-41_SOD81_P10.16mm_Horizontal, F.Cu at (92.1, 131.4)
- added D8: D, Diode_THT:D_DO-41_SOD81_P10.16mm_Horizontal, F.Cu at (99.7, 131.4)
- added D9: D, Diode_THT:D_DO-41_SOD81_P10.16mm_Horizontal, F.Cu at (118.5, 131.4)
- added J39: Leak sensors, Connector_PinHeader_2.54mm:PinHeader_1x04_P2.54mm_Vertical, F.Cu at (201.3, 103.8)
- added J40: Leak sensors, Connector_PinHeader_2.54mm:PinHeader_1x04_P2.54mm_Vertical, F.Cu at (401.3, 103.8)
- added J41: TA_C, Connector_PinHeader_2.54mm:PinHeader_1x01_P2.54mm_Vertical, F.Cu at (387.7, 91.0)
- added J42: TB_C, Connector_PinHeader_2.54mm:PinHeader_1x01_P2.54mm_Vertical, F.Cu at (387.7, 97.7)
- added J43: TC_C, Connector_PinHeader_2.54mm:PinHeader_1x01_P2.54mm_Vertical, F.Cu at (387.7, 105.3)
- added J44: TD_C, Connector_PinHeader_2.54mm:PinHeader_1x01_P2.54mm_Vertical, F.Cu at (387.7, 112.8)
- added J45: TB_C, Connector_PinHeader_2.54mm:PinHeader_1x01_P2.54mm_Vertical, F.Cu at (187.7, 97.7)
- added J46: TC_C, Connector_PinHeader_2.54mm:PinHeader_1x01_P2.54mm_Vertical, F.Cu at (187.7, 105.3)
- added J47: TD_C, Connector_PinHeader_2.54mm:PinHeader_1x01_P2.54mm_Vertical, F.Cu at (187.7, 112.8)
- added J48: S3 S5 LEDs, Connector_PinHeader_2.54mm:PinHeader_1x02_P2.54mm_Vertical, F.Cu at (372.6, 98.7)
- added J49: S1 S2 LEDs, Connector_PinHeader_2.54mm:PinHeader_1x02_P2.54mm_Vertical, F.Cu at (169.9, 98.9)
- added J50: S1 S2 BTNS, Connector_PinHeader_2.54mm:PinHeader_1x02_P2.54mm_Vertical, F.Cu at (172.6, 98.9)
- added J51: U17 IN, Connector_PinHeader_2.54mm:PinHeader_1x02_P2.54mm_Vertical, F.Cu at (69.8, 68.8)
- added J52: U8 IN, Connector_PinHeader_2.54mm:PinHeader_1x02_P2.54mm_Vertical, F.Cu at (130.2, 68.8)
- added J53: X0 IN, Connector_PinHeader_2.54mm:PinHeader_1x02_P2.54mm_Vertical, F.Cu at (169.8, 68.8)
- added J54: X9 IN, Connector_PinHeader_2.54mm:PinHeader_1x02_P2.54mm_Vertical, F.Cu at (230.2, 68.8)
- added Q10: MMBT3904, Package_TO_SOT_SMD:SOT-23, B.Cu at (186.7, 116.5)
- added Q5: IRF4905, Package_TO_SOT_THT:TO-220-3_Vertical, F.Cu at (121.3, 123.5)
- added Q6: IRF4905, Package_TO_SOT_THT:TO-220-3_Vertical, F.Cu at (128.8, 123.5)
- added Q7: MMBT3904, Package_TO_SOT_SMD:SOT-23, B.Cu at (186.7, 93.8)
- added Q8: MMBT3904, Package_TO_SOT_SMD:SOT-23, B.Cu at (186.7, 101.5)
- added Q9: MMBT3904, Package_TO_SOT_SMD:SOT-23, B.Cu at (186.7, 109.1)
- added R16: R, Resistor_SMD:R_1206_3216Metric, B.Cu at (227.7, 72.5)
- added R32: R, Resistor_SMD:R_1206_3216Metric, B.Cu at (196.6, 76.6)
- added R33: R, Resistor_SMD:R_1206_3216Metric, B.Cu at (202.3, 76.6)
- added R34: R, Resistor_SMD:R_1206_3216Metric, B.Cu at (208.0, 76.6)
- added R35: R, Resistor_SMD:R_1206_3216Metric, B.Cu at (213.7, 76.6)
- added R36: 1k, Resistor_SMD:R_0805_2012Metric, B.Cu at (369.8, 106.5)
- added R37: 1k, Resistor_SMD:R_0805_2012Metric, B.Cu at (369.8, 93.6)
- added R38: R, Resistor_SMD:R_1206_3216Metric, B.Cu at (169.8, 72.5)
- added R40: 8.2k, Resistor_SMD:R_0805_2012Metric, B.Cu at (131.3, 123.0)
- added R41: 5.1k, Resistor_SMD:R_0805_2012Metric, B.Cu at (123.9, 128.0)
- added R42: 5.1k, Resistor_SMD:R_0805_2012Metric, B.Cu at (131.3, 128.0)
- added R43: 1k, Resistor_SMD:R_0805_2012Metric, B.Cu at (390.0, 88.0)
- added R44: 1k, Resistor_SMD:R_0805_2012Metric, B.Cu at (390.0, 97.0)
- added R45: 1k, Resistor_SMD:R_0805_2012Metric, B.Cu at (390.0, 103.0)
- added R46: 1k, Resistor_SMD:R_0805_2012Metric, B.Cu at (390.0, 112.0)
- added R47: 1k, Resistor_SMD:R_0805_2012Metric, B.Cu at (395.0, 88.0)
- added R48: 1k, Resistor_SMD:R_0805_2012Metric, B.Cu at (395.0, 97.0)
- added R49: 1k, Resistor_SMD:R_0805_2012Metric, B.Cu at (395.0, 103.0)
- added R50: 1k, Resistor_SMD:R_0805_2012Metric, B.Cu at (395.0, 112.0)
- added R51: R, Resistor_SMD:R_0805_2012Metric, B.Cu at (190.7, 94.6)
- added R52: R, Resistor_SMD:R_0805_2012Metric, B.Cu at (190.7, 102.3)
- added R53: R, Resistor_SMD:R_0805_2012Metric, B.Cu at (190.7, 109.9)
- added R54: R, Resistor_SMD:R_0805_2012Metric, B.Cu at (190.7, 117.3)
- added U18: PC817, Package_DIP:DIP-4_W7.62mm, F.Cu at (199.1, 80.0)
- added U19: PC817, Package_DIP:DIP-4_W7.62mm, F.Cu at (204.8, 80.0)
- added U20: PC817, Package_DIP:DIP-4_W7.62mm, F.Cu at (210.5, 80.0)
- added U21: PC817, Package_DIP:DIP-4_W7.62mm, F.Cu at (216.2, 80.0)
- added U22: MAX485E, Package_SO:SOIC-8_3.9x4.9mm_P1.27mm, B.Cu at (115.6, 114.4)
- J12: value Display -> S3 S5 LEDs; footprint Connector_PinHeader_2.54mm:PinHeader_1x04_P2.54mm_Vertical -> Connector_PinHeader_2.54mm:PinHeader_1x02_P2.54mm_Vertical
- J17: value Display -> TA_C; footprint Connector_PinHeader_2.54mm:PinHeader_1x04_P2.54mm_Vertical -> Connector_PinHeader_2.54mm:PinHeader_1x01_P2.54mm_Vertical
- R17, R18, R19, R20: value R -> 1k; footprint Resistor_THT:R_Axial_DIN0207_L6.3mm_D2.5mm_P10.16mm_Horizontal -> Resistor_SMD:R_0805_2012Metric; moved to B.Cu
- R27, R28: value R -> 820; footprint Resistor_SMD:R_1206_3216Metric -> Resistor_SMD:R_0805_2012Metric
- R29: value R -> 8.2k; footprint Resistor_SMD:R_1206_3216Metric -> Resistor_SMD:R_0805_2012Metric
- moved R19 225.6 mm to (426.5, 92.5)
- moved R17 203.6 mm to (405.0, 92.5), turned to 180 degrees
- moved R20 196.3 mm to (426.5, 107.5), turned to 0 degrees
- moved R18 175.0 mm to (405.0, 107.5)
- moved U17 115.1 mm to (172.3, 76.0)
- moved U8 100.2 mm to (230.2, 76.0)
- moved R29 43.7 mm to (123.9, 123.0)
- moved D4 43.1 mm to (390.0, 115.0)
- moved J13 30.1 mm to (127.5, 104.5), turned to 180 degrees
- moved J22 29.7 mm to (227.5, 103.8), turned to 180 degrees
- moved D3 26.4 mm to (390.0, 106.0)
- moved S2 25.8 mm to (376.5, 89.5), turned to 90 degrees
- moved R27 20.4 mm to (124.3, 106.3), turned to -90 degrees
- moved J17 19.2 mm to (187.7, 91.0), turned to 0 degrees
- moved J11 17.8 mm to (75.9, 106.1), turned to 90 degrees
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Connections:
- D1 pad 1: unconnected-(D1-Pad1) -> Net-(D1-Pad1)
- D1 pad 2: unconnected-(D1-Pad2) -> /Top board/VDD
- D1 pad 3: unconnected-(D1-Pad3) -> Net-(D1-Pad3)
- D2 pad 1: unconnected-(D2-Pad1) -> Net-(D2-Pad1)
- D2 pad 2: unconnected-(D2-Pad2) -> /Top board/VDD
- D2 pad 3: unconnected-(D2-Pad3) -> Net-(D2-Pad3)
- D3 pad 1: unconnected-(D3-Pad1) -> Net-(D3-Pad1)
- D3 pad 2: unconnected-(D3-Pad2) -> /Top board/VDD
- D3 pad 3: unconnected-(D3-Pad3) -> Net-(D3-Pad3)
- D4 pad 1: unconnected-(D4-Pad1) -> Net-(D4-Pad1)
- D4 pad 2: unconnected-(D4-Pad2) -> /Top board/VDD
- D4 pad 3: unconnected-(D4-Pad3) -> Net-(D4-Pad3)
- J11 pad 1: /PB7 -> /PB0
- J11 pad 2: /PB6 -> /PB1
- J11 pad 3: /PB5 -> /PB2
- J11 pad 4: /PB4 -> /PB3
- J12 pad 1: /Top board/GND -> /Top board/S2LED
- J12 pad 2: /Top board/VCC -> /Top board/S1LED
- J17 pad 1: /Middle board/GND -> Net-(J17-Pad1)
- J18 pad 1: /Middle board/PB7 -> /Middle board/S1LED
- J18 pad 3: /Middle board/PB5 -> /Middle board/S2BTN
- J18 pad 4: /Middle board/PB4 -> /Middle board/S2LED
- J19 pad 1: /PD2 -> unconnected-(J19-Pad1)
- J19 pad 2: /PD3 -> unconnected-(J19-Pad2)
- J19 pad 3: /PD4 -> unconnected-(J19-Pad3)
- J19 pad 4: /PD5 -> unconnected-(J19-Pad4)
- J21 pad 1: unconnected-(J21-Pad1) -> /Middle board/SD
- J21 pad 2: unconnected-(J21-Pad2) -> /Middle board/SC
- J21 pad 3: unconnected-(J21-Pad3) -> /Middle board/SB
- J21 pad 4: unconnected-(J21-Pad4) -> /Middle board/SA
- J25 pad 1: /Middle board/S3LED -> /Middle board/PD3
- J25 pad 2: /Middle board/S5LED -> /Middle board/PD2
- J26 pad 1: /Middle board/S4LED -> /Middle board/PD4
- J26 pad 2: /Middle board/S6LED -> /Middle board/PD5
- J31 pad 1: /Middle board/PC7 -> /Middle board/PC4
- J32 pad 1: /Middle board/PC4 -> /Middle board/PC5
- J33 pad 1: /Middle board/PC6 -> /Middle board/PC7
- J34 pad 1: /Middle board/PC5 -> /Middle board/PC6
- J36 pad 1: unconnected-(J36-Pad1) -> /Middle board/S_B
- J36 pad 2: unconnected-(J36-Pad2) -> /Middle board/S_A
- J37 pad 1: unconnected-(J37-Pad1) -> /Middle board/S_D
- J37 pad 2: unconnected-(J37-Pad2) -> /Middle board/S_C
- J5 pad 1: unconnected-(J5-Pad1) -> /Y4
- J5 pad 2: unconnected-(J5-Pad2) -> /Y5
- R10 pad 1: /Q3 -> /PB7
- R17 pad 1: /Middle board/S3LED -> /Top board/S3LED
- R17 pad 2: /Middle board/PD2 -> Net-(R17-Pad2)
- R18 pad 1: /Middle board/S4LED -> /Top board/S5LED
- R18 pad 2: /Middle board/PD3 -> Net-(R18-Pad2)
- R19 pad 1: /Middle board/S5LED -> /Top board/S4LED
- R19 pad 2: /Middle board/PD4 -> Net-(R19-Pad2)
- R20 pad 1: /Middle board/S6LED -> /Top board/S6LED
- R20 pad 2: /Middle board/PD5 -> Net-(R20-Pad2)
- R27 pad 1: unconnected-(R27-Pad1) -> /PD6
- R28 pad 1: unconnected-(R28-Pad1) -> /PD7
- R29 pad 1: unconnected-(R29-Pad1) -> Net-(R29-Pad1)
- R29 pad 2: Net-(U8-Pad2) -> Net-(Q5-Pad1)
- R3 pad 1: /Q0 -> /PB4
- R4 pad 1: /Q1 -> /PB5
- R7 pad 1: /Q2 -> /PB6
- S1 pad 1: unconnected-(S1-Pad1) -> /Top board/S1BTN
- S1 pad 2: unconnected-(S1-Pad2) -> /Top board/S1BTN
- S1 pad 3: unconnected-(S1-Pad3) -> /Top board/VSS
- S1 pad 4: unconnected-(S1-Pad4) -> /Top board/VSS
- S1 pad A: unconnected-(S1-PadA) -> Net-(S1-PadA)
- S1 pad C: unconnected-(S1-PadC) -> /Top board/VSS
- S2 pad 1: unconnected-(S2-Pad1) -> /Top board/S2BTN
- S2 pad 2: unconnected-(S2-Pad2) -> /Top board/S2BTN
- S2 pad 3: unconnected-(S2-Pad3) -> /Top board/VSS
- S2 pad 4: unconnected-(S2-Pad4) -> /Top board/VSS
- S2 pad A: unconnected-(S2-PadA) -> Net-(S2-PadA)
- S2 pad C: unconnected-(S2-PadC) -> /Top board/VSS
- S3 pad 3: /Top board/GND -> /Top board/VSS
- S3 pad 4: /Top board/GND -> /Top board/VSS
- S3 pad A: /Top board/S3LED -> Net-(R17-Pad2)
- S3 pad C: /Top board/GND -> /Top board/VSS
- S4 pad 3: /Top board/GND -> /Top board/VSS
- S4 pad 4: /Top board/GND -> /Top board/VSS
- S4 pad A: /Top board/S4LED -> Net-(R19-Pad2)
- S4 pad C: /Top board/GND -> /Top board/VSS
- S5 pad 3: /Top board/GND -> /Top board/VSS
- S5 pad 4: /Top board/GND -> /Top board/VSS
- S5 pad A: /Top board/S5LED -> Net-(R18-Pad2)
- S5 pad C: /Top board/GND -> /Top board/VSS
- S6 pad 3: /Top board/GND -> /Top board/VSS
- S6 pad 4: /Top board/GND -> /Top board/VSS
- S6 pad A: /Top board/S6LED -> Net-(R20-Pad2)
- S6 pad C: /Top board/GND -> /Top board/VSS
- U1 pad 1: /Q0 -> /PB0
- U1 pad 14: /PD0 -> /RXD
- U1 pad 15: /PD1 -> /TXD
- U1 pad 18: unconnected-(U1-Pad18) -> /PD4
- U1 pad 19: unconnected-(U1-Pad19) -> /PD5
- U1 pad 2: /Q1 -> /PB1
- U1 pad 20: unconnected-(U1-Pad20) -> /PD6
- U1 pad 21: unconnected-(U1-Pad21) -> /PD7
- U1 pad 24: unconnected-(U1-Pad24) -> /PC2
- U1 pad 25: unconnected-(U1-Pad25) -> /PC3
- U1 pad 3: /Q2 -> /PB2
- U1 pad 4: /Q3 -> /PB3
- U17 pad 1: /VCC -> /Middle board/VCC
- U17 pad 2: unconnected-(U17-Pad2) -> Net-(R38-Pad2)
- U17 pad 3: /VSS -> /Middle board/VSS
- U17 pad 4: /PA0 -> unconnected-(U17-Pad4)
- U6 pad 1: /VCC -> /VDD
- U6 pad 3: /VSS -> /GND
- U6 pad 4: unconnected-(U6-Pad4) -> Net-(R29-Pad1)
- U7 pad 1: /VCC -> /VDD
- U7 pad 3: /VSS -> /GND
- U7 pad 4: unconnected-(U7-Pad4) -> Net-(R40-Pad1)
- U8 pad 1: /VCC -> /Middle board/VCC
- U8 pad 2: Net-(U8-Pad2) -> Net-(R16-Pad2)
- U8 pad 3: /VSS -> /Middle board/VSS
Routing:
- net /Top board/VSS: track 0.00 -> 172.7 mm
- net /Top board/GND: track 100.8 -> 0.00 mm
- net /Middle board/SD: track 0.00 -> 78.6 mm, vias 0 -> 2
- net /Middle board/SC: track 0.00 -> 58.5 mm, vias 0 -> 2
- net /Middle board/VSS: track 0.00 -> 49.9 mm, vias 0 -> 4
- net /Middle board/SB: track 0.00 -> 44.4 mm, vias 0 -> 2
- net /Middle board/PC5: track 46.6 -> 2.71 mm
- net /Middle board/VCC: track 0.00 -> 39.5 mm, vias 0 -> 4
- net /VCC: track 136.9 -> 170.9 mm, vias 7 -> 0
- net /PC7: track 2.56 -> 35.3 mm
- net /Middle board/PC6: track 34.0 -> 2.71 mm
- net /Top board/VDD: track 0.00 -> 30.0 mm
- net /GND: track 56.4 -> 86.3 mm, vias 7 -> 1
- net /Middle board/SA: track 0.00 -> 29.4 mm, vias 0 -> 2
- net /PC6: track 2.56 -> 31.3 mm
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
Commit message: update
Parts:
- removed H5, H6, H7: MountingHole, MountingHole:MountingHole_3.2mm_M3
- removed the R16 at (227.7, 72.5)
- removed the R16 at (63.4, 90.1)
- added 22pF1: C, Capacitor_SMD:C_0805_2012Metric, B.Cu at (103.9, 101.5)
- added 22pF2: C, Capacitor_SMD:C_0805_2012Metric, B.Cu at (109.3, 112.8)
- added BZ1: Buzzer, Buzzer_Beeper:Buzzer_12x9.5RM7.6, F.Cu at (74.2, 110.1)
- added C1: C, Capacitor_SMD:C_0805_2012Metric, B.Cu at (100.0, 86.2)
- added C2: C_Polarized, Capacitor_SMD:C_1812_4532Metric, B.Cu at (219.8, 115.8)
- added J55: AVR-ISP-10, Connector_IDC:IDC-Header_2x05_P2.54mm_Vertical, B.Cu at (96.2, 98.5)
- added J56: U17 OUT, Connector_PinHeader_2.54mm:PinHeader_1x02_P2.54mm_Vertical, B.Cu at (172.3, 91.0)
- added J57: U8 OUT, Connector_PinHeader_2.54mm:PinHeader_1x02_P2.54mm_Vertical, B.Cu at (227.6, 86.0)
- added J58: U17 OUT, Connector_PinHeader_2.54mm:PinHeader_1x02_P2.54mm_Vertical, F.Cu at (72.3, 91.0)
- added J59: U8 OUT, Connector_PinHeader_2.54mm:PinHeader_1x02_P2.54mm_Vertical, F.Cu at (127.6, 86.0)
- added J60: GND, Connector_PinHeader_2.54mm:PinHeader_1x01_P2.54mm_Vertical, B.Cu at (171.9, 69.6)
- added J61: GND, Connector_PinHeader_2.54mm:PinHeader_1x01_P2.54mm_Vertical, F.Cu at (71.9, 69.6)
- added J62: VCC, Connector_PinHeader_2.54mm:PinHeader_1x01_P2.54mm_Vertical, B.Cu at (188.7, 71.1)
- added J63: VCC, Connector_PinHeader_2.54mm:PinHeader_1x01_P2.54mm_Vertical, F.Cu at (88.7, 71.1)
- added J64: SIM800, Connector_PinHeader_2.54mm:PinHeader_1x06_P2.54mm_Vertical, F.Cu at (206.8, 130.0)
- added J65: RES_IN, TerminalBlock_Phoenix:TerminalBlock_Phoenix_MKDS-1,5-2-5.08_1x02_P5.08mm_Horizontal, F.Cu at (177.1, 127.9)
- added J66: SELF_PWR_IN, TerminalBlock_Phoenix:TerminalBlock_Phoenix_MKDS-1,5-2-5.08_1x02_P5.08mm_Horizontal, F.Cu at (217.7, 127.9)
- added J67: VDD VSS, Connector_PinHeader_2.54mm:PinHeader_1x02_P2.54mm_Vertical, B.Cu at (416.3, 118.7)
- added J68: VDD VSS, Connector_PinHeader_2.54mm:PinHeader_1x02_P2.54mm_Vertical, F.Cu at (216.3, 118.7)
- added J69: VDD, Connector_PinHeader_2.54mm:PinHeader_1x01_P2.54mm_Vertical, F.Cu at (130.2, 103.8)
- added J70: VDD, Connector_PinHeader_2.54mm:PinHeader_1x01_P2.54mm_Vertical, B.Cu at (230.2, 103.8)
- added J71: RES_OUT, Connector_PinHeader_2.54mm:PinHeader_1x01_P2.54mm_Vertical, F.Cu at (170.2, 107.3)
- added J72: VSS, Connector_PinHeader_2.54mm:PinHeader_1x01_P2.54mm_Vertical, F.Cu at (181.0, 112.4)
- added J73: VSS, Connector_PinHeader_2.54mm:PinHeader_1x01_P2.54mm_Vertical, F.Cu at (181.5, 81.5)
- added J74: VSS, Connector_PinHeader_2.54mm:PinHeader_1x01_P2.54mm_Vertical, F.Cu at (223.4, 81.5)
- added J75: VSS, Connector_PinHeader_2.54mm:PinHeader_1x01_P2.54mm_Vertical, B.Cu at (423.4, 81.5)
- added J76: VSS, Connector_PinHeader_2.54mm:PinHeader_1x01_P2.54mm_Vertical, B.Cu at (381.5, 81.5)
- added J77: VDD, Connector_PinHeader_2.54mm:PinHeader_1x01_P2.54mm_Vertical, F.Cu at (182.5, 118.7)
- added J78: VDD, Connector_PinHeader_2.54mm:PinHeader_1x01_P2.54mm_Vertical, B.Cu at (382.5, 118.7)
- added J79: NC, Connector_PinHeader_2.54mm:PinHeader_1x01_P2.54mm_Vertical, B.Cu at (169.5, 130.5)
- added J80: NC, Connector_PinHeader_2.54mm:PinHeader_1x01_P2.54mm_Vertical, F.Cu at (69.5, 130.5)
- added J81: NC, Connector_PinHeader_2.54mm:PinHeader_1x01_P2.54mm_Vertical, F.Cu at (113.5, 130.5)
- added J82: NC, Connector_PinHeader_2.54mm:PinHeader_1x01_P2.54mm_Vertical, B.Cu at (213.5, 130.5)
- added JP1: Dir Control, Jumper:SolderJumper-3_P1.3mm_Bridged2Bar12_Pad1.0x1.5mm, B.Cu at (110.2, 101.2)
- added R16: R, Resistor_SMD:R_1206_3216Metric, B.Cu at (227.6, 72.5)
- added R39: 820, Resistor_SMD:R_0805_2012Metric, B.Cu at (110.2, 92.4)
- added R55: 820, Resistor_SMD:R_0805_2012Metric, B.Cu at (110.2, 90.5)
- added R56: 820, Resistor_SMD:R_0805_2012Metric, B.Cu at (110.3, 79.8)
- added R57: 820, Resistor_SMD:R_0805_2012Metric, B.Cu at (104.5, 79.8)
- added R58: 820, Resistor_SMD:R_0805_2012Metric, B.Cu at (98.8, 79.8)
- added R59: 820, Resistor_SMD:R_0805_2012Metric, B.Cu at (74.2, 87.5)
- added R60: 820, Resistor_SMD:R_0805_2012Metric, B.Cu at (130.2, 83.0)
- added R61: 1k, Resistor_SMD:R_0805_2012Metric, B.Cu at (103.9, 99.5)
- added R62: R, Resistor_SMD:R_0805_2012Metric, B.Cu at (179.7, 109.2)
- added R63: R, Resistor_THT:R_Axial_DIN0309_L9.0mm_D3.2mm_P5.08mm_Vertical, F.Cu at (170.0, 122.9)
- added U23: PC817, Package_DIP:DIP-4_W7.62mm, F.Cu at (173.4, 118.7)
- J10: value X_INS -> AUX_INS
- J12, J16, J18, J20, J21, J22, J23, J24, J27, J28, J29, J30, J40, J41, J42, J43, J44, J48, J54: moved to B.Cu
- J51: value U17 IN -> X0; footprint Connector_PinHeader_2.54mm:PinHeader_1x02_P2.54mm_Vertical -> Connector_PinHeader_2.54mm:PinHeader_1x01_P2.54mm_Vertical; moved to B.Cu
- J53: value X0 IN -> X0; footprint Connector_PinHeader_2.54mm:PinHeader_1x02_P2.54mm_Vertical -> Connector_PinHeader_2.54mm:PinHeader_1x01_P2.54mm_Vertical
- moved J53 100.4 mm to (69.4, 69.6), turned to 0 degrees
- moved J51 99.6 mm to (169.4, 69.6), turned to 180 degrees
- moved R14 7.52 mm to (79.8, 83.1)
- moved R13 5.52 mm to (92.8, 79.8)
- moved R15 4.38 mm to (74.2, 83.1), turned to 180 degrees
- moved R38 2.54 mm to (169.8, 75.0)
- moved U17 2.54 mm to (172.3, 78.5)
- moved J13 0.74 mm to (127.5, 103.8)
- turned J12 to 180 degrees
- turned J16 to 90 degrees
- turned J18 to -90 degrees
- turned J20 to -90 degrees
- turned J21 to -90 degrees
- turned J22 to 0 degrees
- turned J23 to 180 degrees
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Connections:
- net /Middle board/S1LED renamed /Middle board/PB7
- net /Middle board/S2BTN renamed /Middle board/PB5
- net /Middle board/S2LED renamed /Middle board/PB4
- J35 pad 1: unconnected-(J35-Pad1) -> /Middle board/VCC
- J35 pad 2: unconnected-(J35-Pad2) -> /Middle board/GND
- J38 pad 1: unconnected-(J38-Pad1) -> /Middle board/VCC
- J38 pad 2: unconnected-(J38-Pad2) -> /Middle board/GND
- J4 pad 1: unconnected-(J4-Pad1) -> /B
- J4 pad 2: unconnected-(J4-Pad2) -> /A
- J51 pad 1: /X0 -> /Middle board/X0
- J53 pad 1: /Middle board/X0 -> /X0
- U1 pad 11: Net-(U1-Pad11) -> /VSS
- U1 pad 30: unconnected-(U1-Pad30) -> /VDD
- U1 pad 31: Net-(U1-Pad11) -> /VSS
- U1 pad 32: unconnected-(U1-Pad32) -> /VDD
- U1 pad 9: unconnected-(U1-Pad9) -> /RST
- U10 pad 4: unconnected-(U10-Pad4) -> /PC4
- U11 pad 4: unconnected-(U11-Pad4) -> /PC5
- U12 pad 4: unconnected-(U12-Pad4) -> /PC6
- U13 pad 4: unconnected-(U13-Pad4) -> /PC7
- U17 pad 4: unconnected-(U17-Pad4) -> /Middle board/PA0
- U22 pad 2: unconnected-(U22-Pad2) -> Net-(JP1-Pad2)
- U22 pad 3: unconnected-(U22-Pad3) -> Net-(JP1-Pad2)
- U22 pad 5: unconnected-(U22-Pad5) -> /VSS
- U22 pad 6: unconnected-(U22-Pad6) -> /A
- U22 pad 7: unconnected-(U22-Pad7) -> /B
- U22 pad 8: unconnected-(U22-Pad8) -> /VDD
- U8 pad 4: unconnected-(U8-Pad4) -> /Middle board/PC2
- U9 pad 4: unconnected-(U9-Pad4) -> /PC3
Routing:
- net /Middle board/VSS: track 49.9 -> 253.2 mm, vias 4 -> 7
- net /VSS: track 51.6 -> 214.4 mm
- net /VDD: track 64.2 -> 209.4 mm, vias 4 -> 11
- net /Middle board/VDD: track 0.00 -> 115.7 mm, vias 0 -> 2
- net /Middle board/SCL: track 0.00 -> 61.2 mm, vias 0 -> 2
- net /VCC: track 170.9 -> 231.0 mm
- net /SDA: track 2.54 -> 61.3 mm
- net /GND: track 86.3 -> 143.4 mm
- net /Middle board/GND: track 0.00 -> 52.6 mm
- net /Middle board/SDA: track 0.00 -> 51.4 mm, vias 0 -> 2
- net /Middle board/VCC: track 39.5 -> 86.2 mm, vias 4 -> 7
- net /Top board/VDD: track 30.0 -> 65.8 mm
- net /Top board/VSS: track 172.7 -> 208.5 mm
- net /B: track 0.00 -> 24.7 mm
- net /A: track 0.00 -> 24.4 mm
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- added copper zone on B.Cu, net /Top board/VSS
- added copper zone on B.Cu, net /VSS
Other:
- outline, holes or cut-outs redrawn
- board text added: "(c) 2023 semicontinuity"
- board text added: "0V"
- board text added: "24V"
- board text added: "5V POWER SUPPLY"
- board text added: "A"
- board text added: "AUX INPUTS"
- board text added: "AUX OUTPUTS"
- board text added: "B"
- board text added: "CONTROLLER"
- board text added: "GND"
- board text added: "MAX485/MAX13487"
- board text added: "Optional"
- board text added: "POWER FOR SENSORS"
- board text added: "QC:"
- board text added: "R"
- board text added: "RS485"
- board text added: "SIM800 optional"
- board text added: "VALVE CONTROL INPUTS"
- board text added: "VALVE STATE INPUTS"
- board text added: "VCC"
- board text added: "VDD"
- board text added: "VSS"
- board text added: "Valve outputs"
- board text added: "WATER LEAK SENSORS"
- board text added: "optional DC/DC 24->5V"
- board text added: "v1.0"

Commit message: plc-4u-a += pcb update
Parts:
- added C3: C, Capacitor_SMD:C_0805_2012Metric, B.Cu at (99.8, 86.0)
- J71: value RES_OUT -> RESERVED_OUT
- moved C1 19.4 mm to (100.5, 105.5), turned to 0 degrees
Connections:
- net /Middle board/SDA renamed /Middle board/RXD
Routing:
- net /VSS: track 214.4 -> 230.8 mm, vias 0 -> 1
- net /VDD: track 209.4 -> 203.0 mm, vias 11 -> 12
- net unconnected-(J19-Pad4): track 2.40 -> 0.00 mm
- net unconnected-(J19-Pad2): track 0.00 -> 2.40 mm
- net unconnected-(J19-Pad1): track 2.40 -> 0.00 mm
- net /PD5: track 0.00 -> 2.40 mm
- net /PD3: track 2.40 -> 0.00 mm
- net /PD2: track 0.00 -> 2.40 mm

Commit message: plc-4u-a board += leds
Parts:
- added D11: LED, LED_THT:LED_D3.0mm, F.Cu at (208.8, 116.3)
- added D12: LED, LED_THT:LED_D3.0mm, F.Cu at (201.7, 117.6)
- added H5: MountingHole, MountingHole:MountingHole_3.2mm_M3, F.Cu at (186.5, 75.5)
- added H6: MountingHole, MountingHole:MountingHole_3.2mm_M3, F.Cu at (214.5, 124.5)
- added J83: RXD, Connector_PinHeader_2.54mm:PinHeader_1x01_P2.54mm_Vertical, F.Cu at (113.2, 110.8)
- added J84: RXD, Connector_PinHeader_2.54mm:PinHeader_1x01_P2.54mm_Vertical, B.Cu at (213.2, 110.8)
- added J85: TXD, Connector_PinHeader_2.54mm:PinHeader_1x01_P2.54mm_Vertical, F.Cu at (118.5, 110.8)
- added J86: TXD, Connector_PinHeader_2.54mm:PinHeader_1x01_P2.54mm_Vertical, B.Cu at (218.5, 110.8)
- added R64: R, Resistor_SMD:R_0805_2012Metric, B.Cu at (216.8, 113.6)
- added R65: R, Resistor_SMD:R_0805_2012Metric, B.Cu at (209.8, 110.8)
- moved C2 5.00 mm to (219.8, 120.8)
- moved U22 1.00 mm to (115.6, 115.4)
- moved J52 0.50 mm to (130.2, 69.3)
- moved J54 0.50 mm to (230.2, 69.3)
Connections:
- net /Middle board/RXD renamed /Middle board/RX
- J19 pad 1: unconnected-(J19-Pad1) -> /PD2
- J19 pad 2: unconnected-(J19-Pad2) -> /PD3
- J19 pad 3: unconnected-(J19-Pad3) -> /PD4
- J19 pad 4: unconnected-(J19-Pad4) -> /PD5
Routing:
- net /Top board/S6BTN: track 5.45 -> 17.9 mm
- net /Top board/S5BTN: track 3.40 -> 15.9 mm
- net /Top board/S4BTN: track 5.45 -> 17.9 mm
- net /Top board/S3BTN: track 3.40 -> 15.9 mm
- net /Middle board/RX: track 51.4 -> 62.5 mm
- net Net-(R65-Pad2): track 0.00 -> 10.5 mm
- net /Top board/VSS: track 208.5 -> 198.1 mm
- net /Top board/VDD: track 65.8 -> 75.6 mm
- net Net-(R64-Pad2): track 0.00 -> 8.22 mm
- net /Middle board/VSS: track 253.2 -> 259.4 mm, vias 7 -> 8
- net /Middle board/SCL: track 61.2 -> 56.9 mm
- net /Middle board/TXD: track 0.00 -> 3.46 mm
- net /VDD: track 203.0 -> 206.4 mm
- net /Middle board/RXD: track 0.00 -> 2.56 mm
- net /Middle board/VDD: track 115.7 -> 118.2 mm
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- removed copper zone on B.Cu, net /Top board/VSS
Other:
- outline, holes or cut-outs redrawn
